File: KiCad/FreeEEG32.kicad_pcb (KiCad board)
At the start: 4 copper layers, 70 x 70 mm, 183 parts, among them P1 CONN_02X10, P11 CONN_01X03, P2 CONN_02X10, P3 CONN_02X10, P4 CONN_02X10, P5 CONN_01X02, P6 CONN_01X06, P7 CONN_01X06, P8 USB_B, SW1 NRST, SW2 SWITCH_INV, SW3 SWITCH_INV, T1 da2303, U1 ADP7118AUJZ-3.3_TSOT, U10 TPD4E1B06, U11 TPD4E1B06, U12 TPD4E1B06, U13 AD7770, U14 ADR4525, U15 TPD4E1B06, U16 TPD4E1B06, U17 TPD4E1B06, U18 TPD4E1B06, U19 TPD4E1B06, U2 ADP7118AUJZ-3.3_TSOT, U20 AD7770, U21 ADR4525, U22 TPD4E1B06, U23 TPD4E1B06, U24 TPD4E1B06, U25 TPD4E1B06, U26 TPD4E1B06, U27 AD7770, U28 ADR4525, U29 TPD4E1B06, U3 8.192MHz, U30 TPD4E1B06, U31 TPD4E1B06, U32 TPD4E1B06, U33 TPD4E1B06, U34 AD7770, U35 ISO7342c_uart, U36 ISO7341c_spi, U37 STM32F427ZI_4side_short, U38 LP5907_WIFI, U39 ADP7118AUJZ-3.3_TSOT, U40 CP2102N-24, U41 MPU-6500, U42 LP5912, U43 473521001, U5 ESP-12E, U6 SN6505A, U7 ADR4525, U8 TPD4E1B06, U9 TPD4E1B06, Y1 32.768kHz, Y2 8MHz

Commit message: kicad
Parts:
- added C118: 100n, Capacitors_SMD:C_0402, B.Cu at (-11.0, -6.50)
- C3, C4, U41: moved to F.Cu
- P8: footprint Connect:USB_Micro-B -> usb_b_circular:USB_Micro-B_circular
- U14, U21, U28, U7: moved to B.Cu
- U5: value ESP-12E -> ESP-12F
- Y2: footprint Crystals:Crystal_SMD_5032-4pin_5.0x3.2mm -> Crystals:Crystal_SMD_5032_4Pads; moved to F.Cu
- moved U39 55.8 mm to (-11.4, -11.4), turned to 315 degrees
- moved U1 41.8 mm to (-11.4, 11.4), turned to 45 degrees
- moved U40 38.7 mm to (-19.1, -20.3)
- moved C1 36.4 mm to (0.80, 81.5)
- moved C2 36.4 mm to (0.80, 81.5)
- moved C5 36.4 mm to (0.80, 81.5)
- moved P5 36.4 mm to (0.80, 81.5)
- moved R1 36.4 mm to (0.80, 81.5)
- moved SW1 36.4 mm to (0.80, 81.5)
- moved U12 36.4 mm to (0.80, 81.5)
- moved U19 36.4 mm to (0.80, 81.5)
- moved U26 36.4 mm to (0.80, 81.5)
- moved U33 36.4 mm to (0.80, 81.5)
- moved Y1 36.4 mm to (0.80, 81.5)
- moved U38 32.4 mm to (-22.9, -33.7), turned to 315 degrees
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Connections:
- U37 pad 10: Net-(U37-Pad10) -> AD3_DRDY
- U37 pad 11: Net-(U37-Pad11) -> AD3_START
- U37 pad 118: Net-(U37-Pad118) -> AD2_DRDY
- U37 pad 119: Net-(U37-Pad119) -> AD2_START
- U37 pad 126: Net-(U37-Pad126) -> AD2_RESET
- U37 pad 15: Net-(U37-Pad15) -> AD3_RESET
- U37 pad 46: Net-(U37-Pad46) -> AD4_DRDY
- U37 pad 47: Net-(U37-Pad47) -> AD4_START
- U37 pad 54: Net-(U37-Pad54) -> AD4_RESET
- U37 pad 79: Net-(U37-Pad79) -> AD1_DRDY
- U37 pad 83: Net-(U37-Pad83) -> GND
- U37 pad 84: Net-(U37-Pad84) -> VDD
- U37 pad 85: Net-(U37-Pad85) -> AD1_START
- U37 pad 90: Net-(U37-Pad90) -> AD1_RESET
Routing:
- net IOVDD: track 26.7 -> 115.6 mm, vias 5 -> 10
- net V+: track 10.9 -> 63.5 mm, vias 3 -> 7
- net UART_TX_USB: track 5.52 -> 44.7 mm
- net UART_RX_USB: track 5.99 -> 44.0 mm
- net GND: track 295.7 -> 320.7 mm, vias 9 -> 14
- net SPI6_NSS: track 0.00 -> 24.9 mm, vias 0 -> 1
- net USART1_TX: track 0.00 -> 18.3 mm
- net USART1_RX: track 0.00 -> 12.8 mm
- net SPI6_MISO: track 0.00 -> 12.2 mm, vias 0 -> 1
- net USART1_CTS: track 0.00 -> 12.1 mm
- net USART1_RTS: track 0.00 -> 11.3 mm
- net D+_USB: track 0.80 -> 10.6 mm
- net AD3_RESET: track 0.00 -> 9.29 mm, vias 0 -> 1
- net AD2_RESET: track 0.00 -> 8.76 mm, vias 0 -> 1
- net AD4_RESET: track 0.00 -> 8.71 mm, vias 0 -> 1
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
Commit message: kicad & restructure catalogs
Parts:
- moved U38 69.6 mm to (-86.4, -62.1)
- moved C112 36.7 mm to (-70.8, 71.7)
- moved R2 36.7 mm to (-67.8, 81.0)
- moved C109 36.7 mm to (-70.3, 77.5)
- moved C110 36.7 mm to (-64.6, 78.9)
- moved C111 36.7 mm to (-74.3, 81.2)
- moved SW2 36.7 mm to (-77.5, 74.6)
- moved P11 29.1 mm to (86.4, -51.8)
- moved C117 28.9 mm to (-80.7, -68.2)
- moved C116 28.9 mm to (-80.5, -65.8)
- moved C24 28.9 mm to (-74.2, -74.8)
- moved C25 28.9 mm to (-70.5, -77.8)
- moved U42 28.9 mm to (-78.0, -69.7)
- moved REF** 27.3 mm to (78.8, -74.9)
- moved C103 1.08 mm to (-15.0, 3.75)
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Connections:
- U37 pad 122: Net-(U37-Pad122) -> AD2_RESET
- U37 pad 126: AD2_RESET -> Net-(U37-Pad126)
Routing:
- net SDIO_D0: track 0.00 -> 33.0 mm, vias 0 -> 3
- net SDIO_D1: track 0.00 -> 32.9 mm, vias 0 -> 3
- net SPI6_NSS: track 24.9 -> 0.00 mm, vias 1 -> 0
- net SPI6_MISO: track 12.2 -> 0.00 mm, vias 1 -> 0
- net GND: track 320.7 -> 328.9 mm, vias 14 -> 13
- net SPI6_MOSI: track 6.37 -> 0.00 mm, vias 1 -> 0
- net SPI6_SCK: track 6.33 -> 0.00 mm, vias 1 -> 0
- net VDD: track 27.9 -> 31.7 mm, vias 2 -> 1
- net Net-(C103-Pad2): track 0.33 -> 2.34 mm
- net AD2_RESET: track 8.76 -> 7.81 mm

Commit message: kicad
Parts:
- removed C1: CL1, Capacitors_SMD:C_0402
- removed C116: 10u, Capacitors_SMD:C_0402
- removed C117: 1u, Capacitors_SMD:C_0402
- removed C2: CL2, Capacitors_SMD:C_0402
- removed C5: 100n, Capacitors_SMD:C_0402
- removed P5: CONN_01X02, Socket_Strips:Socket_Strip_Straight_1x02
- removed R1: REXT, Resistors_SMD:R_0402
- removed the REF** at (78.8, -74.9)
- removed U12, U19, U26, U33: TPD4E1B06, TO_SOT_Packages_SMD:SC-70-6
- removed U42: LP5912, WSON-6_2x2mm_Pitch0.65mm:WSON-6_2x2mm_Pitch0.65mm
- removed Y1: 32.768kHz, Crystals:Crystal_SMD_0603_2Pads_obsolete
- SW1, U41: moved to B.Cu
- U5: moved to F.Cu
- moved C25 124.9 mm to (-16.6, 34.9)
- moved C24 124.5 mm to (-18.4, 36.5)
- moved SW2 122.3 mm to (-20.4, -33.5), turned to 225 degrees
- moved C111 117.1 mm to (-31.5, -27.8)
- moved U38 116.8 mm to (-19.4, 33.6)
- moved C110 115.3 mm to (-25.1, -29.4)
- moved R2 115.3 mm to (-28.3, -27.4)
- moved C109 115.3 mm to (-30.9, -30.8)
- moved C112 112.5 mm to (-28.1, -32.5)
- moved SW3 108.9 mm to (-33.5, -20.9), turned to 225 degrees
- moved SW1 107.8 mm to (32.9, -21.5), turned to 225 degrees
- moved U5 80.7 mm to (-35.8, 35.2)
- moved P11 65.3 mm to (25.4, -28.3)
- moved U41 8.98 mm to (19.7, -19.7)
- moved C101 2.57 mm to (-13.5, 5.25), turned to 45 degrees
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Routing:
- net (no net): track 1.82 -> 77.2 mm
- net AD1_SYNC_IN: track 2.33 -> 63.4 mm, vias 0 -> 4
- net SPI6_NSS: track 0.00 -> 47.1 mm, vias 0 -> 2
- net SDIO_DETECT: track 0.00 -> 46.3 mm, vias 0 -> 1
- net UART_TX_USB: track 44.7 -> 5.52 mm
- net UART_RX_USB: track 44.0 -> 5.99 mm
- net SDIO_D2: track 0.00 -> 27.2 mm, vias 0 -> 1
- net SDIO_D3: track 0.00 -> 25.6 mm, vias 0 -> 1
- net SDIO_CK: track 0.00 -> 24.2 mm, vias 0 -> 1
- net SPI6_SCK: track 0.00 -> 23.7 mm, vias 0 -> 2
- net SPI6_MOSI: track 0.00 -> 21.0 mm
- net VDD: track 31.7 -> 48.7 mm, vias 1 -> 4
- net GND: track 328.9 -> 345.0 mm, vias 13 -> 15
- net SDIO_CMD: track 0.00 -> 15.7 mm, vias 0 -> 1
- net SPI6_MISO: track 0.00 -> 15.2 mm
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
Commit message: kicad
Parts:
- removed R2: 1k, Resistors_SMD:R_0402
- removed REF**: SW_DIP_x8_W5.08mm_Slide_Copal_CHS-A, Buttons_Switches_SMD:SW_DIP_x8_W5.08mm_Slide_Copal_CHS-A
- removed REF**: SW_DIP_x8_W6.15mm_Slide_Omron_A6H, Buttons_Switches_SMD:SW_DIP_x8_W6.15mm_Slide_Omron_A6H
- removed REF**: SW_DIP_x8_W7.62mm_Slide_Copal_CHS-B, Buttons_Switches_SMD:SW_DIP_x8_W7.62mm_Slide_Copal_CHS-B
- removed U38: LP5907_WIFI, TO_SOT_Packages_SMD:SOT-23-5
- added C1: 100n, Capacitors_SMD:C_0402, B.Cu at (5.00, 15.9)
- added C116: 1u, Capacitors_SMD:C_0402, B.Cu at (5.25, 14.6)
- added C117: 2.2u, Capacitors_SMD:C_0603, F.Cu at (-13.5, -12.4)
- added C119: 2.2u, Capacitors_SMD:C_0603, F.Cu at (-10.0, 10.9)
- added C120: 2.2u, Capacitors_SMD:C_0603, F.Cu at (14.2, 15.2)
- added C121: 2.2u, Capacitors_SMD:C_0603, F.Cu at (-9.53, -10.5)
- added C122: 2.2u, Capacitors_SMD:C_0603, F.Cu at (-7.87, 6.99)
- added C123: 2.2u, Capacitors_SMD:C_0603, F.Cu at (11.4, 12.4)
- added C124: 2.2u, Capacitors_SMD:C_0603, B.Cu at (-4.57, -14.1)
- added C2: 1u, Capacitors_SMD:C_0402, B.Cu at (5.50, 16.4)
- added C5: 100n, Capacitors_SMD:C_0402, B.Cu at (4.75, 14.1)
- added U19: TLV73333PDBVT, TO_SOT_Packages_SMD:SOT-23-5, B.Cu at (-26.7, 17.8)
- C102, C106, C111, C112, C113, C114: footprint Capacitors_SMD:C_0402 -> Capacitors_SMD:C_0603
- C24: value 1u -> 100n; moved to B.Cu
- C25, P8: moved to B.Cu
- P6, P7: value CONN_01X06 -> CONN_02X03; footprint Socket_Strips:Socket_Strip_Straight_1x06 -> Socket_Strips:Socket_Strip_Straight_2x03
- SW2, SW3: footprint Buttons_Switches_SMD:SW_SPDT_PCM12 -> Buttons_Switches_SMD:SW_SPST_B3U-1100P-B; moved to B.Cu
- moved SW3 54.5 mm to (-15.2, 30.5), turned to 315 degrees
- moved SW2 54.1 mm to (30.5, -15.2), turned to 135 degrees
- moved D3 34.3 mm to (-27.3, -16.5)
- moved C24 22.7 mm to (-29.2, 16.5)
- moved C112 20.5 mm to (-17.4, -15.1)
- moved C109 20.2 mm to (-19.6, -13.9), turned to 225 degrees
- moved C25 20.1 mm to (-24.8, 16.5), turned to 315 degrees
- moved U5 19.6 mm to (-21.6, 21.6)
- moved C111 17.4 mm to (-20.2, -14.5), turned to 225 degrees
- moved C110 17.1 mm to (-16.9, -14.5)
- moved P11 11.7 mm to (14.0, -26.0), turned to 45 degrees
- moved C4 6.29 mm to (6.30, 11.6), turned to 45 degrees
- moved C3 6.21 mm to (11.1, 6.85), turned to 225 degrees
- moved SW1 5.83 mm to (27.3, -19.7), turned to 315 degrees
- moved C115 4.07 mm to (-12.1, 10.8), turned to 135 degrees
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- renumbered U41 to U12
Connections:
- net Net-(C109-Pad1) renamed VDD_USB
- net Net-(U37-Pad69) renamed I2C2_SCL
- net Net-(U37-Pad70) renamed I2C2_SDA
- C102 pad 1: VDD -> Net-(C102-Pad1)
- C103 pad 2: Net-(C103-Pad2) -> VDD
- C24 pad 1: GND_WIFI -> GND_ISO_UART
- C24 pad 2: V+_WIFI -> V+_ISO_UART
- C25 pad 1: GND_WIFI -> GND_ISO_UART
- C7 pad 1: GND -> VDD
- C7 pad 2: VDD -> GND
- P1 pad 19: Net-(P1-Pad19) -> GND
- P1 pad 2: Net-(P1-Pad2) -> Net-(P1-Pad1)
- P1 pad 20: Net-(P1-Pad20) -> GND
- P2 pad 19: Net-(P2-Pad19) -> GND
- P2 pad 2: Net-(P2-Pad2) -> Net-(P2-Pad1)
- P2 pad 20: Net-(P2-Pad20) -> GND
- P3 pad 19: Net-(P3-Pad19) -> GND
- P3 pad 2: Net-(P3-Pad2) -> Net-(P3-Pad1)
- P3 pad 20: Net-(P3-Pad20) -> GND
- P4 pad 19: Net-(P4-Pad19) -> GND
- P4 pad 2: Net-(P4-Pad2) -> Net-(P4-Pad1)
- P4 pad 20: Net-(P4-Pad20) -> GND
- SW2 pad 1: Net-(R2-Pad2) -> GND
- SW2 pad 2: RSTb_USB -> VDD
- SW2 pad 3: GND_ISO_UART -> BOOT0
- SW3 pad 2: CH_PD_WIFI -> GND_ISO_UART
- SW3 pad 3: GND_WIFI -> BOOT_WIFI
- U1 pad 4: Net-(U1-Pad4) -> AVDD
- U10 pad 3: /ADC1/VSS -> GND
- U11 pad 3: /ADC1/VSS -> GND
- U13 pad 17: /ADC1/CONVST_SAR -> GND
- U15 pad 3: /ADC2/VSS -> GND
- U16 pad 3: /ADC2/VSS -> GND
- U17 pad 3: /ADC2/VSS -> GND
- U18 pad 3: /ADC2/VSS -> GND
- U2 pad 4: Net-(U2-Pad4) -> IOVDD
- U20 pad 17: /ADC2/CONVST_SAR -> GND
- U22 pad 3: /ADC3/VSS -> GND
- U23 pad 3: /ADC3/VSS -> GND
- U24 pad 3: /ADC3/VSS -> GND
- U25 pad 3: /ADC3/VSS -> GND
- U27 pad 17: /ADC3/CONVST_SAR -> GND
- U29 pad 3: /ADC4/VSS -> GND
- U30 pad 3: /ADC4/VSS -> GND
- U31 pad 3: /ADC4/VSS -> GND
- U32 pad 3: /ADC4/VSS -> GND
- U34 pad 17: /ADC4/CONVST_SAR -> GND
- U37 pad 100: SDIO_DETECT -> Net-(U37-Pad100)
- U37 pad 25: NRST -> Net-(U37-Pad25)
- U37 pad 27: Net-(U37-Pad27) -> NRST
- U37 pad 30: GND -> VDD
- U37 pad 31: VDD -> GND
- U37 pad 32: Net-(U37-Pad32) -> VDD
- U37 pad 33: Net-(U37-Pad33) -> VDD
- U37 pad 6: Net-(U37-Pad6) -> VDD
- U37 pad 71: VDD -> Net-(C102-Pad1)
- U37 pad 72: Net-(C103-Pad2) -> VDD
- U37 pad 97: Net-(U37-Pad97) -> SDIO_DETECT
- U39 pad 4: Net-(U39-Pad4) -> VDD
- U43 pad 1: SDIO_D2 -> Net-(U43-Pad1)
- U5 pad 15: GND_WIFI -> GND_ISO_UART
- U5 pad 17: Net-(U5-Pad17) -> VCC_WIFI
- U5 pad 18: Net-(U5-Pad18) -> BOOT_WIFI
- U5 pad 3: CH_PD_WIFI -> VCC_WIFI
- U8 pad 3: /ADC1/VSS -> GND
- U9 pad 3: /ADC1/VSS -> GND
Routing:
- net GND: track 345.0 -> 595.6 mm, vias 15 -> 40
- net GND_ISO_UART: track 37.1 -> 142.0 mm, vias 1 -> 4
- net UART_CTS_USB: track 5.46 -> 88.3 mm, vias 0 -> 2
- net (no net): track 77.2 -> 0.00 mm
- net UART_RTS_USB: track 6.04 -> 80.9 mm, vias 0 -> 2
- net VDD: track 48.7 -> 122.4 mm, vias 4 -> 5
- net NRST: track 0.00 -> 68.0 mm, vias 0 -> 2
- net V+_ISO_UART: track 31.3 -> 98.1 mm, vias 1 -> 2
- net Net-(P1-Pad1): track 0.00 -> 64.2 mm
- net UART_TX_USB: track 5.52 -> 61.6 mm
- net Net-(P2-Pad1): track 0.00 -> 55.1 mm
- net Net-(P3-Pad1): track 0.00 -> 54.0 mm
- net D-_USB: track 6.73 -> 60.3 mm, vias 0 -> 1
- net D+_USB: track 10.6 -> 62.0 mm, vias 0 -> 1
- net UART_RX_USB: track 5.99 -> 56.6 mm
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
Commit message: kicad
Parts:
- U35: value ISO7342c_uart -> ADUM1402BRWZ
Connections:
- C13 pad 1: /ADC1/REF1+ -> /ADC4/REF1+
- C17 pad 1: /ADC1/REF1+ -> /ADC4/REF1+
- C21 pad 2: /ADC1/REF1+ -> /ADC4/REF1+
- C30 pad 2: /ADC1/REF1+ -> /ADC4/REF1+
- C34 pad 2: /ADC1/REF_OUT -> /ADC4/REF_OUT
- C36 pad 1: /ADC2/REF1+ -> /ADC1/REF1+
- C40 pad 1: /ADC2/REF1+ -> /ADC1/REF1+
- C45 pad 2: /ADC2/REF1+ -> /ADC1/REF1+
- C53 pad 2: /ADC2/REF1+ -> /ADC1/REF1+
- C57 pad 2: /ADC2/REF_OUT -> /ADC1/REF_OUT
- C59 pad 1: /ADC3/REF1+ -> /ADC2/REF1+
- C63 pad 1: /ADC3/REF1+ -> /ADC2/REF1+
- C67 pad 2: /ADC3/REF1+ -> /ADC2/REF1+
- C74 pad 2: /ADC3/REF1+ -> /ADC2/REF1+
- C78 pad 2: /ADC3/REF_OUT -> /ADC2/REF_OUT
- C80 pad 1: /ADC4/REF1+ -> /ADC3/REF1+
- C84 pad 1: /ADC4/REF1+ -> /ADC3/REF1+
- C88 pad 2: /ADC4/REF1+ -> /ADC3/REF1+
- C95 pad 2: /ADC4/REF1+ -> /ADC3/REF1+
- C99 pad 2: /ADC4/REF_OUT -> /ADC3/REF_OUT
- P1 pad 10: /ADC1/AIN3+ -> /ADC4/AIN3+
- P1 pad 11: /ADC1/AIN4- -> /ADC4/AIN4-
- P1 pad 12: /ADC1/AIN4+ -> /ADC4/AIN4+
- P1 pad 13: /ADC1/AIN5- -> /ADC4/AIN5-
- P1 pad 14: /ADC1/AIN5+ -> /ADC4/AIN5+
- P1 pad 15: /ADC1/AIN6- -> /ADC4/AIN6-
- P1 pad 16: /ADC1/AIN6+ -> /ADC4/AIN6+
- P1 pad 17: /ADC1/AIN7- -> /ADC4/AIN7-
- P1 pad 18: /ADC1/AIN7+ -> /ADC4/AIN7+
- P1 pad 3: /ADC1/AIN0- -> /ADC4/AIN0-
- P1 pad 4: /ADC1/AIN0+ -> /ADC4/AIN0+
- P1 pad 5: /ADC1/AIN1- -> /ADC4/AIN1-
- P1 pad 6: /ADC1/AIN1+ -> /ADC4/AIN1+
- P1 pad 7: /ADC1/AIN2- -> /ADC4/AIN2-
- P1 pad 8: /ADC1/AIN2+ -> /ADC4/AIN2+
- P1 pad 9: /ADC1/AIN3- -> /ADC4/AIN3-
- P2 pad 10: /ADC2/AIN3+ -> /ADC1/AIN3+
- P2 pad 11: /ADC2/AIN4- -> /ADC1/AIN4-
- P2 pad 12: /ADC2/AIN4+ -> /ADC1/AIN4+
- P2 pad 13: /ADC2/AIN5- -> /ADC1/AIN5-
- P2 pad 14: /ADC2/AIN5+ -> /ADC1/AIN5+
- P2 pad 15: /ADC2/AIN6- -> /ADC1/AIN6-
- P2 pad 16: /ADC2/AIN6+ -> /ADC1/AIN6+
- P2 pad 17: /ADC2/AIN7- -> /ADC1/AIN7-
- P2 pad 18: /ADC2/AIN7+ -> /ADC1/AIN7+
- P2 pad 3: /ADC2/AIN0- -> /ADC1/AIN0-
- P2 pad 4: /ADC2/AIN0+ -> /ADC1/AIN0+
- P2 pad 5: /ADC2/AIN1- -> /ADC1/AIN1-
- P2 pad 6: /ADC2/AIN1+ -> /ADC1/AIN1+
- P2 pad 7: /ADC2/AIN2- -> /ADC1/AIN2-
- P2 pad 8: /ADC2/AIN2+ -> /ADC1/AIN2+
- P2 pad 9: /ADC2/AIN3- -> /ADC1/AIN3-
- P3 pad 10: /ADC3/AIN3+ -> /ADC2/AIN3+
- P3 pad 11: /ADC3/AIN4- -> /ADC2/AIN4-
- P3 pad 12: /ADC3/AIN4+ -> /ADC2/AIN4+
- P3 pad 13: /ADC3/AIN5- -> /ADC2/AIN5-
- P3 pad 14: /ADC3/AIN5+ -> /ADC2/AIN5+
- P3 pad 15: /ADC3/AIN6- -> /ADC2/AIN6-
- P3 pad 16: /ADC3/AIN6+ -> /ADC2/AIN6+
- P3 pad 17: /ADC3/AIN7- -> /ADC2/AIN7-
- P3 pad 18: /ADC3/AIN7+ -> /ADC2/AIN7+
- P3 pad 3: /ADC3/AIN0- -> /ADC2/AIN0-
- P3 pad 4: /ADC3/AIN0+ -> /ADC2/AIN0+
- P3 pad 5: /ADC3/AIN1- -> /ADC2/AIN1-
- P3 pad 6: /ADC3/AIN1+ -> /ADC2/AIN1+
- P3 pad 7: /ADC3/AIN2- -> /ADC2/AIN2-
- P3 pad 8: /ADC3/AIN2+ -> /ADC2/AIN2+
- P3 pad 9: /ADC3/AIN3- -> /ADC2/AIN3-
- P4 pad 10: /ADC4/AIN3+ -> /ADC3/AIN3+
- P4 pad 11: /ADC4/AIN4- -> /ADC3/AIN4-
- P4 pad 12: /ADC4/AIN4+ -> /ADC3/AIN4+
- P4 pad 13: /ADC4/AIN5- -> /ADC3/AIN5-
- P4 pad 14: /ADC4/AIN5+ -> /ADC3/AIN5+
- P4 pad 15: /ADC4/AIN6- -> /ADC3/AIN6-
- P4 pad 16: /ADC4/AIN6+ -> /ADC3/AIN6+
- P4 pad 17: /ADC4/AIN7- -> /ADC3/AIN7-
- P4 pad 18: /ADC4/AIN7+ -> /ADC3/AIN7+
- P4 pad 3: /ADC4/AIN0- -> /ADC3/AIN0-
- P4 pad 4: /ADC4/AIN0+ -> /ADC3/AIN0+
- P4 pad 5: /ADC4/AIN1- -> /ADC3/AIN1-
- P4 pad 6: /ADC4/AIN1+ -> /ADC3/AIN1+
- P4 pad 7: /ADC4/AIN2- -> /ADC3/AIN2-
- P4 pad 8: /ADC4/AIN2+ -> /ADC3/AIN2+
- P4 pad 9: /ADC4/AIN3- -> /ADC3/AIN3-
- P6 pad 2: UART_RX_USB -> UART_TX_USB
- P6 pad 3: UART_CTS_USB -> UART_RTS_USB
- P6 pad 4: UART_TX_USB -> UART_RX_USB
- P6 pad 5: UART_RTS_USB -> UART_CTS_USB
- U10 pad 1: /ADC1/AIN5+ -> /ADC4/AIN5+
- U10 pad 2: /ADC1/AIN5- -> /ADC4/AIN5-
- U10 pad 4: /ADC1/AIN4- -> /ADC4/AIN4-
- U10 pad 5: /ADC1/AIN4+ -> /ADC4/AIN4+
- U11 pad 1: /ADC1/AIN7+ -> /ADC4/AIN7+
- U11 pad 2: /ADC1/AIN7- -> /ADC4/AIN7-
- U11 pad 4: /ADC1/AIN6- -> /ADC4/AIN6-
- U11 pad 5: /ADC1/AIN6+ -> /ADC4/AIN6+
- U13 pad 1: /ADC1/AIN0- -> /ADC4/AIN0-
- U13 pad 10: /ADC1/AIN2+ -> /ADC4/AIN2+
- U13 pad 11: /ADC1/AIN3- -> /ADC4/AIN3-
- U13 pad 12: /ADC1/AIN3+ -> /ADC4/AIN3+
- U13 pad 13: /ADC1/GPIO0 -> /ADC4/GPIO0
- U13 pad 14: /ADC1/GPIO1 -> /ADC4/GPIO1
- U13 pad 15: /ADC1/GPIO2 -> /ADC4/GPIO2
- U13 pad 16: /ADC1/ALERT -> /ADC4/ALERT
- U13 pad 2: /ADC1/AIN0+ -> /ADC4/AIN0+
- U13 pad 25: /ADC1/DOUT3 -> /ADC4/DOUT3
- U13 pad 26: /ADC1/DOUT2 -> /ADC4/DOUT2
- U13 pad 27: /ADC1/DOUT1 -> /ADC4/DOUT1
- U13 pad 28: /ADC1/DOUT0 -> /ADC4/DOUT0
- U13 pad 29: /ADC1/DCLK -> /ADC4/DCLK
- U13 pad 3: /ADC1/AIN1- -> /ADC4/AIN1-
- U13 pad 37: /ADC1/AIN7+ -> /ADC4/AIN7+
- U13 pad 38: /ADC1/AIN7- -> /ADC4/AIN7-
- U13 pad 39: /ADC1/AIN6+ -> /ADC4/AIN6+
- U13 pad 4: /ADC1/AIN1+ -> /ADC4/AIN1+
- U13 pad 40: /ADC1/AIN6- -> /ADC4/AIN6-
- U13 pad 41: /ADC1/REF1+ -> /ADC4/REF1+
- U13 pad 45: /ADC1/AIN5+ -> /ADC4/AIN5+
- U13 pad 46: /ADC1/AIN5- -> /ADC4/AIN5-
- U13 pad 47: /ADC1/AIN4+ -> /ADC4/AIN4+
- U13 pad 48: /ADC1/AIN4- -> /ADC4/AIN4-
- U13 pad 49: /ADC1/REF_OUT -> /ADC4/REF_OUT
- U13 pad 57: /ADC1/VCM -> /ADC4/VCM
- U13 pad 63: /ADC1/AUXAIN+ -> /ADC4/AUXAIN+
- U13 pad 64: /ADC1/AUXAIN- -> /ADC4/AUXAIN-
- U13 pad 8: /ADC1/REF1+ -> /ADC4/REF1+
- U13 pad 9: /ADC1/AIN2- -> /ADC4/AIN2-
- U14 pad 6: /ADC2/REF1+ -> /ADC1/REF1+
- U15 pad 1: /ADC2/AIN1+ -> /ADC1/AIN1+
- U15 pad 2: /ADC2/AIN1- -> /ADC1/AIN1-
- U15 pad 4: /ADC2/AIN0- -> /ADC1/AIN0-
- U15 pad 5: /ADC2/AIN0+ -> /ADC1/AIN0+
- U16 pad 1: /ADC2/AIN3+ -> /ADC1/AIN3+
- U16 pad 2: /ADC2/AIN3- -> /ADC1/AIN3-
- U16 pad 4: /ADC2/AIN2- -> /ADC1/AIN2-
- U16 pad 5: /ADC2/AIN2+ -> /ADC1/AIN2+
- U17 pad 1: /ADC2/AIN5+ -> /ADC1/AIN5+
- U17 pad 2: /ADC2/AIN5- -> /ADC1/AIN5-
- U17 pad 4: /ADC2/AIN4- -> /ADC1/AIN4-
- U17 pad 5: /ADC2/AIN4+ -> /ADC1/AIN4+
- U18 pad 1: /ADC2/AIN7+ -> /ADC1/AIN7+
- U18 pad 2: /ADC2/AIN7- -> /ADC1/AIN7-
- U18 pad 4: /ADC2/AIN6- -> /ADC1/AIN6-
- U18 pad 5: /ADC2/AIN6+ -> /ADC1/AIN6+
- U20 pad 1: /ADC2/AIN0- -> /ADC1/AIN0-
- U20 pad 10: /ADC2/AIN2+ -> /ADC1/AIN2+
- U20 pad 11: /ADC2/AIN3- -> /ADC1/AIN3-
- U20 pad 12: /ADC2/AIN3+ -> /ADC1/AIN3+
- U20 pad 13: /ADC2/GPIO0 -> /ADC1/GPIO0
- U20 pad 14: /ADC2/GPIO1 -> /ADC1/GPIO1
- U20 pad 15: /ADC2/GPIO2 -> /ADC1/GPIO2
- U20 pad 16: /ADC2/ALERT -> /ADC1/ALERT
- U20 pad 2: /ADC2/AIN0+ -> /ADC1/AIN0+
- U20 pad 25: /ADC2/DOUT3 -> /ADC1/DOUT3
- U20 pad 26: /ADC2/DOUT2 -> /ADC1/DOUT2
- U20 pad 27: /ADC2/DOUT1 -> /ADC1/DOUT1
- U20 pad 28: /ADC2/DOUT0 -> /ADC1/DOUT0
- U20 pad 29: /ADC2/DCLK -> /ADC1/DCLK
- U20 pad 3: /ADC2/AIN1- -> /ADC1/AIN1-
- U20 pad 37: /ADC2/AIN7+ -> /ADC1/AIN7+
- U20 pad 38: /ADC2/AIN7- -> /ADC1/AIN7-
- U20 pad 39: /ADC2/AIN6+ -> /ADC1/AIN6+
- U20 pad 4: /ADC2/AIN1+ -> /ADC1/AIN1+
- U20 pad 40: /ADC2/AIN6- -> /ADC1/AIN6-
- U20 pad 41: /ADC2/REF1+ -> /ADC1/REF1+
- U20 pad 45: /ADC2/AIN5+ -> /ADC1/AIN5+
- U20 pad 46: /ADC2/AIN5- -> /ADC1/AIN5-
- U20 pad 47: /ADC2/AIN4+ -> /ADC1/AIN4+
- U20 pad 48: /ADC2/AIN4- -> /ADC1/AIN4-
- U20 pad 49: /ADC2/REF_OUT -> /ADC1/REF_OUT
- U20 pad 57: /ADC2/VCM -> /ADC1/VCM
- U20 pad 63: /ADC2/AUXAIN+ -> /ADC1/AUXAIN+
- U20 pad 64: /ADC2/AUXAIN- -> /ADC1/AUXAIN-
- U20 pad 8: /ADC2/REF1+ -> /ADC1/REF1+
- U20 pad 9: /ADC2/AIN2- -> /ADC1/AIN2-
- U21 pad 6: /ADC3/REF1+ -> /ADC2/REF1+
- U22 pad 1: /ADC3/AIN1+ -> /ADC2/AIN1+
- U22 pad 2: /ADC3/AIN1- -> /ADC2/AIN1-
- U22 pad 4: /ADC3/AIN0- -> /ADC2/AIN0-
- U22 pad 5: /ADC3/AIN0+ -> /ADC2/AIN0+
- U23 pad 1: /ADC3/AIN3+ -> /ADC2/AIN3+
- U23 pad 2: /ADC3/AIN3- -> /ADC2/AIN3-
- U23 pad 4: /ADC3/AIN2- -> /ADC2/AIN2-
- U23 pad 5: /ADC3/AIN2+ -> /ADC2/AIN2+
- U24 pad 1: /ADC3/AIN5+ -> /ADC2/AIN5+
- U24 pad 2: /ADC3/AIN5- -> /ADC2/AIN5-
- U24 pad 4: /ADC3/AIN4- -> /ADC2/AIN4-
- U24 pad 5: /ADC3/AIN4+ -> /ADC2/AIN4+
- U25 pad 1: /ADC3/AIN7+ -> /ADC2/AIN7+
- U25 pad 2: /ADC3/AIN7- -> /ADC2/AIN7-
- U25 pad 4: /ADC3/AIN6- -> /ADC2/AIN6-
- U25 pad 5: /ADC3/AIN6+ -> /ADC2/AIN6+
- U27 pad 1: /ADC3/AIN0- -> /ADC2/AIN0-
- U27 pad 10: /ADC3/AIN2+ -> /ADC2/AIN2+
- U27 pad 11: /ADC3/AIN3- -> /ADC2/AIN3-
- U27 pad 12: /ADC3/AIN3+ -> /ADC2/AIN3+
- U27 pad 13: /ADC3/GPIO0 -> /ADC2/GPIO0
- U27 pad 14: /ADC3/GPIO1 -> /ADC2/GPIO1
- U27 pad 15: /ADC3/GPIO2 -> /ADC2/GPIO2
- U27 pad 16: /ADC3/ALERT -> /ADC2/ALERT
- U27 pad 2: /ADC3/AIN0+ -> /ADC2/AIN0+
- U27 pad 25: /ADC3/DOUT3 -> /ADC2/DOUT3
- U27 pad 26: /ADC3/DOUT2 -> /ADC2/DOUT2
- U27 pad 27: /ADC3/DOUT1 -> /ADC2/DOUT1
- U27 pad 28: /ADC3/DOUT0 -> /ADC2/DOUT0
- U27 pad 29: /ADC3/DCLK -> /ADC2/DCLK
- U27 pad 3: /ADC3/AIN1- -> /ADC2/AIN1-
- U27 pad 37: /ADC3/AIN7+ -> /ADC2/AIN7+
- U27 pad 38: /ADC3/AIN7- -> /ADC2/AIN7-
- U27 pad 39: /ADC3/AIN6+ -> /ADC2/AIN6+
- U27 pad 4: /ADC3/AIN1+ -> /ADC2/AIN1+
- U27 pad 40: /ADC3/AIN6- -> /ADC2/AIN6-
- U27 pad 41: /ADC3/REF1+ -> /ADC2/REF1+
- U27 pad 45: /ADC3/AIN5+ -> /ADC2/AIN5+
- U27 pad 46: /ADC3/AIN5- -> /ADC2/AIN5-
- U27 pad 47: /ADC3/AIN4+ -> /ADC2/AIN4+
- U27 pad 48: /ADC3/AIN4- -> /ADC2/AIN4-
- U27 pad 49: /ADC3/REF_OUT -> /ADC2/REF_OUT
- U27 pad 57: /ADC3/VCM -> /ADC2/VCM
- U27 pad 63: /ADC3/AUXAIN+ -> /ADC2/AUXAIN+
- U27 pad 64: /ADC3/AUXAIN- -> /ADC2/AUXAIN-
- U27 pad 8: /ADC3/REF1+ -> /ADC2/REF1+
- U27 pad 9: /ADC3/AIN2- -> /ADC2/AIN2-
- U28 pad 6: /ADC4/REF1+ -> /ADC3/REF1+
- U29 pad 1: /ADC4/AIN1+ -> /ADC3/AIN1+
- U29 pad 2: /ADC4/AIN1- -> /ADC3/AIN1-
- U29 pad 4: /ADC4/AIN0- -> /ADC3/AIN0-
- U29 pad 5: /ADC4/AIN0+ -> /ADC3/AIN0+
- U30 pad 1: /ADC4/AIN3+ -> /ADC3/AIN3+
- U30 pad 2: /ADC4/AIN3- -> /ADC3/AIN3-
- U30 pad 4: /ADC4/AIN2- -> /ADC3/AIN2-
- U30 pad 5: /ADC4/AIN2+ -> /ADC3/AIN2+
- U31 pad 1: /ADC4/AIN5+ -> /ADC3/AIN5+
- U31 pad 2: /ADC4/AIN5- -> /ADC3/AIN5-
- U31 pad 4: /ADC4/AIN4- -> /ADC3/AIN4-
- U31 pad 5: /ADC4/AIN4+ -> /ADC3/AIN4+
- U32 pad 1: /ADC4/AIN7+ -> /ADC3/AIN7+
- U32 pad 2: /ADC4/AIN7- -> /ADC3/AIN7-
- U32 pad 4: /ADC4/AIN6- -> /ADC3/AIN6-
- U32 pad 5: /ADC4/AIN6+ -> /ADC3/AIN6+
- U34 pad 1: /ADC4/AIN0- -> /ADC3/AIN0-
- U34 pad 10: /ADC4/AIN2+ -> /ADC3/AIN2+
- U34 pad 11: /ADC4/AIN3- -> /ADC3/AIN3-
- U34 pad 12: /ADC4/AIN3+ -> /ADC3/AIN3+
- U34 pad 13: /ADC4/GPIO0 -> /ADC3/GPIO0
- U34 pad 14: /ADC4/GPIO1 -> /ADC3/GPIO1
- U34 pad 15: /ADC4/GPIO2 -> /ADC3/GPIO2
- U34 pad 16: /ADC4/ALERT -> /ADC3/ALERT
- U34 pad 2: /ADC4/AIN0+ -> /ADC3/AIN0+
- U34 pad 25: /ADC4/DOUT3 -> /ADC3/DOUT3
- U34 pad 26: /ADC4/DOUT2 -> /ADC3/DOUT2
- U34 pad 27: /ADC4/DOUT1 -> /ADC3/DOUT1
- U34 pad 28: /ADC4/DOUT0 -> /ADC3/DOUT0
- U34 pad 29: /ADC4/DCLK -> /ADC3/DCLK
- U34 pad 3: /ADC4/AIN1- -> /ADC3/AIN1-
- U34 pad 37: /ADC4/AIN7+ -> /ADC3/AIN7+
- U34 pad 38: /ADC4/AIN7- -> /ADC3/AIN7-
- U34 pad 39: /ADC4/AIN6+ -> /ADC3/AIN6+
- U34 pad 4: /ADC4/AIN1+ -> /ADC3/AIN1+
- U34 pad 40: /ADC4/AIN6- -> /ADC3/AIN6-
- U34 pad 41: /ADC4/REF1+ -> /ADC3/REF1+
- U34 pad 45: /ADC4/AIN5+ -> /ADC3/AIN5+
- U34 pad 46: /ADC4/AIN5- -> /ADC3/AIN5-
- U34 pad 47: /ADC4/AIN4+ -> /ADC3/AIN4+
- U34 pad 48: /ADC4/AIN4- -> /ADC3/AIN4-
- U34 pad 49: /ADC4/REF_OUT -> /ADC3/REF_OUT
- U34 pad 57: /ADC4/VCM -> /ADC3/VCM
- U34 pad 63: /ADC4/AUXAIN+ -> /ADC3/AUXAIN+
- U34 pad 64: /ADC4/AUXAIN- -> /ADC3/AUXAIN-
- U34 pad 8: /ADC4/REF1+ -> /ADC3/REF1+
- U34 pad 9: /ADC4/AIN2- -> /ADC3/AIN2-
- U35 pad 3: UART_RX_USB -> UART_TX_USB
- U35 pad 4: UART_CTS_USB -> UART_RTS_USB
- U35 pad 5: UART_TX_USB -> UART_RX_USB
- U35 pad 6: UART_RTS_USB -> UART_CTS_USB
- U40 pad 18: UART_RTS_USB -> UART_CTS_USB
- U40 pad 19: UART_CTS_USB -> UART_RTS_USB
- U40 pad 20: UART_TX_USB -> UART_RX_USB
- U40 pad 21: UART_RX_USB -> UART_TX_USB
- U7 pad 6: /ADC1/REF1+ -> /ADC4/REF1+
- U8 pad 1: /ADC1/AIN1+ -> /ADC4/AIN1+
- U8 pad 2: /ADC1/AIN1- -> /ADC4/AIN1-
- U8 pad 4: /ADC1/AIN0- -> /ADC4/AIN0-
- U8 pad 5: /ADC1/AIN0+ -> /ADC4/AIN0+
- U9 pad 1: /ADC1/AIN3+ -> /ADC4/AIN3+
- U9 pad 2: /ADC1/AIN3- -> /ADC4/AIN3-
- U9 pad 4: /ADC1/AIN2- -> /ADC4/AIN2-
- U9 pad 5: /ADC1/AIN2+ -> /ADC4/AIN2+
Routing:
- net UART_RTS_USB: track 80.9 -> 94.1 mm
- net UART_CTS_USB: track 88.3 -> 93.3 mm
- net UART_RX_USB: track 56.6 -> 61.0 mm
- net /ADC2/AIN6+: track 25.0 -> 23.1 mm
- net D-_USB: track 60.3 -> 62.1 mm
- net D+_USB: track 62.0 -> 63.6 mm
- net /ADC1/AIN6+: track 23.7 -> 25.0 mm
- net /ADC4/REF1+: track 40.2 -> 41.3 mm
- net /ADC1/AIN2-: track 21.8 -> 20.7 mm
- net /ADC4/AIN2-: track 20.8 -> 21.8 mm
- net /ADC2/AIN7-: track 22.6 -> 21.6 mm
- net UART_TX_USB: track 61.6 -> 60.9 mm
- net /ADC1/REF1+: track 41.3 -> 40.6 mm
- net /ADC2/AIN5-: track 14.5 -> 15.2 mm
- net /ADC3/REF1+: track 40.8 -> 40.2 mm
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
Commit message: kicad
Connections:
- U37 pad 25: Net-(U37-Pad25) -> NRST
- U37 pad 27: NRST -> Net-(U37-Pad27)
Routing:
- net NRST: track 68.0 -> 50.5 mm
- net Net-(U37-Pad27): track 0.00 -> 17.1 mm

Commit message: kicad
Changed lines of the file:
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@@
     (links 734)
     (no_connects 27)
-    (area -35.075001 -35.075001 35.075001 35.075001)
+    (area -35.005001 -35.005001 35.005001 35.005001)
     (thickness 1.6)
-    (drawings 47)
+    (drawings 39)
     (tracks 3168)
     (zones 0)
@@
     (trace_min 0.2)
     (segment_width 0.2)
-    (edge_width 0.15)
+    (edge_width 0.001)
     (via_size 0.6)
     (via_drill 0.4)
@@
     (pad "" np_thru_hole circle (at 0 0 315) (size 0.8 0.8) (drill 0.8) (layers *.Cu *.Mask))
   )
+  (gr_line (start -14.49746 -34.99746) (end -34.99746 -14.49746) (angle 90) (layer Edge.Cuts) (width 0.001))
+  (gr_line (start 14.5 -34.99746) (end -14.5 -34.99746) (angle 90) (layer Edge.Cuts) (width 0.001))
   (gr_line (start 0 0) (end 35 0) (angle 90) (layer Cmts.User) (width 0.2))
   (gr_line (start 0 0) (end -34.925 0) (angle 90) (layer Cmts.User) (width 0.2))
@@
   (gr_line (start 0 0) (end 24.765 -24.765) (angle 90) (layer Cmts.User) (width 0.2))
   (gr_circle (center 0 0) (end 2 50) (layer Dwgs.User) (width 0.2))
-  (gr_line (start 14.5 35) (end 35 14.5) (angle 90) (layer Edge.Cuts) (width 0.15))
-  (gr_line (start -14.5 35) (end 14.5 35) (angle 90) (layer Edge.Cuts) (width 0.15))
-  (gr_line (start -35 14.5) (end -14.5 35) (angle 90) (layer Edge.Cuts) (width 0.15))
-  (gr_line (start -35 -14.5) (end -35 14.5) (angle 90) (layer Edge.Cuts) (width 0.15))
-  (gr_line (start -14.5 -35) (end -35 -14.5) (angle 90) (layer Edge.Cuts) (width 0.15))
-  (gr_line (start 14.5 -35) (end -14.5 -35) (angle 90) (layer Edge.Cuts) (width 0.15))
-  (gr_line (start 35 -14.5) (end 14.5 -35) (angle 90) (layer Edge.Cuts) (width 0.15))
-  (gr_line (start 35 14.5) (end 35 -14.5) (angle 90) (layer Edge.Cuts) (width 0.15))
+  (gr_line (start 14.49746 34.99746) (end 34.99746 14.49746) (angle 90) (layer Edge.Cuts) (width 0.001))
+  (gr_line (start -14.5 34.99746) (end 14.5 34.99746) (angle 90) (layer Edge.Cuts) (width 0.001))
+  (gr_line (start -34.99746 14.49746) (end -14.49746 34.99746) (angle 90) (layer Edge.Cuts) (width 0.001))
+  (gr_line (start -34.99746 -14.5) (end -34.99746 14.5) (angle 90) (layer Edge.Cuts) (width 0.001))
+  (gr_line (start 34.99746 -14.49746) (end 14.49746 -34.99746) (angle 90) (layer Edge.Cuts) (width 0.001))
+  (gr_line (start 34.99746 14.5) (end 34.99746 -14.5) (angle 90) (layer Edge.Cuts) (width 0.001))
   (gr_circle (center 0 0) (end 2.54 -19.05) (layer Dwgs.User) (width 0.2))
   (gr_circle (center 0 0) (end 0 -8.89) (layer Dwgs.User) (width 0.2))
@@
   (gr_line (start 0 0) (end 0 -35) (angle 90) (layer Cmts.User) (width 0.2))
   (target plus (at 0 0) (size 5) (width 0.15) (layer Edge.Cuts))
-  (gr_line (start -35 -15) (end -15 -35) (angle 90) (layer Cmts.User) (width 0.2))
-  (gr_line (start -35 15) (end -35 -15) (angle 90) (layer Cmts.User) (width 0.2))
-  (gr_line (start -15 35) (end -35 15) (angle 90) (layer Cmts.User) (width 0.2))
-  (gr_line (start 15 35) (end -15 35) (angle 90) (layer Cmts.User) (width 0.2))
-  (gr_line (start 35 15) (end 15 35) (angle 90) (layer Cmts.User) (width 0.2))
-  (gr_line (start 35 -15) (end 35 15) (angle 90) (layer Cmts.User) (width 0.2))
-  (gr_line (start 15 -35) (end 35 -15) (angle 90) (layer Cmts.User) (width 0.2))
-  (gr_line (start -15 -35) (end 15 -35) (angle 90) (layer Cmts.User) (width 0.2))
   (gr_line (start 35 -35) (end -35 -35) (angle 90) (layer Dwgs.User) (width 0.2))
   (gr_line (start 35 35) (end 35 -35) (angle 90) (layer Dwgs.User) (width 0.2))

Commit message: kicad
Parts:
- added REF**: MountingHole_2.2mm_M2_ISO7380, Mounting_Holes:MountingHole_2.2mm_M2_ISO7380, F.Cu at (28.6, 17.8)
- added REF**: MountingHole_2.2mm_M2_ISO7380, Mounting_Holes:MountingHole_2.2mm_M2_ISO7380, F.Cu at (-28.6, -17.8)
- added REF**: MountingHole_2.2mm_M2_ISO7380, Mounting_Holes:MountingHole_2.2mm_M2_ISO7380, F.Cu at (17.8, 28.6)
- added REF**: MountingHole_2.2mm_M2_ISO7380, Mounting_Holes:MountingHole_2.2mm_M2_ISO7380, F.Cu at (-17.8, -28.6)
- moved D3 2.62 mm to (-24.8, -15.9)
- moved C42 0.64 mm to (-24.8, -17.8)
Routing:
- net Net-(U37-Pad27): track 17.1 -> 0.00 mm
- net NRST: track 50.5 -> 67.6 mm
- net GND_ISO_UART: track 142.0 -> 153.6 mm, vias 4 -> 3
- net V+_ISO_UART: track 98.1 -> 108.5 mm, vias 2 -> 1
- net VCC_WIFI: track 37.9 -> 38.6 mm
- net UART_RX_USB: track 61.0 -> 60.5 mm
