File: KiCad/FreeEEG32.kicad_pcb (KiCad board)
At the start: 4 copper layers, 70 x 70 mm, 181 parts, among them P1 CONN_02X10, P11 CONN_01X03, P2 CONN_02X10, P3 CONN_02X10, P4 CONN_02X10, P6 CONN_02X03, P7 CONN_02X03, P8 USB_B, SW1 NRST, SW2 SWITCH_INV, SW3 SWITCH_INV, T1 da2303, U1 ADP7118AUJZ-3.3_TSOT, U10 TPD4E1B06, U11 TPD4E1B06, U12 MPU-6500, U13 AD7770, U14 ADR4525, U15 TPD4E1B06, U16 TPD4E1B06, U17 TPD4E1B06, U18 TPD4E1B06, U19 TLV73333PDBVT, U2 ADP7118AUJZ-3.3_TSOT, U20 AD7770, U21 ADR4525, U22 TPD4E1B06, U23 TPD4E1B06, U24 TPD4E1B06, U25 TPD4E1B06, U27 AD7770, U28 ADR4525, U29 TPD4E1B06, U3 8.192MHz, U30 TPD4E1B06, U31 TPD4E1B06, U32 TPD4E1B06, U34 AD7770, U35 ADUM1402BRWZ, U36 ISO7341c_spi, U37 STM32F427ZI_4side_short, U39 ADP7118AUJZ-3.3_TSOT, U40 CP2102N-24, U43 473521001, U5 ESP-12F, U6 SN6505A, U7 ADR4525, U8 TPD4E1B06, U9 TPD4E1B06, Y2 8MHz

Commit message: kicad
Parts:
- removed the REF** at (28.6, 17.8)
- removed the REF** at (-28.6, -17.8)
- removed the REF** at (17.8, 28.6)
- removed the REF** at (-17.8, -28.6)
- added C125: 100n, Capacitors_SMD:C_0402, F.Cu at (29.2, -15.2)
- added C126: 100n, Capacitors_SMD:C_0402, F.Cu at (-15.2, 29.2)
- added C127: 100n, Capacitors_SMD:C_0402, B.Cu at (-15.2, 29.2)
- added R1: R_EXT, Resistors_SMD:R_0402, F.Cu at (5.71, 6.60)
- added R2: 47k, Resistors_SMD:R_0402, B.Cu at (29.2, -15.2)
- added R3: 47k, Resistors_SMD:R_0402, B.Cu at (-6.35, 11.4)
- added R4: 47k, Resistors_SMD:R_0402, F.Cu at (-14.2, 28.2)
- added R5: 47k, Resistors_SMD:R_0402, B.Cu at (-14.2, 28.2)
- added R6: 47k, Resistors_SMD:R_0402, F.Cu at (-24.1, 11.4)
- added REF**: MountingHole_2.2mm_M2_ISO7380_Pad, Mounting_Holes:MountingHole_2.2mm_M2_ISO7380_Pad, F.Cu at (-28.6, -17.8)
- added REF**: MountingHole_2.2mm_M2_ISO7380_Pad, Mounting_Holes:MountingHole_2.2mm_M2_ISO7380_Pad, F.Cu at (-17.8, -28.6)
- added REF**: MountingHole_2.2mm_M2_ISO7380_Pad, Mounting_Holes:MountingHole_2.2mm_M2_ISO7380_Pad, F.Cu at (28.6, 17.8)
- added REF**: MountingHole_2.2mm_M2_ISO7380_Pad, Mounting_Holes:MountingHole_2.2mm_M2_ISO7380_Pad, F.Cu at (17.8, 28.6)
- added SW4: BOOT_WIFI, Buttons_Switches_SMD:SW_SPST_B3U-1000P, B.Cu at (-15.9, 31.8)
- SW1: footprint Buttons_Switches_SMD:SW_SPST_B3U-1000P-B -> Buttons_Switches_SMD:SW_SPST_B3U-3000P-B; moved to F.Cu
- SW2: value SWITCH_INV -> BOOT0; footprint Buttons_Switches_SMD:SW_SPST_B3U-1100P-B -> Buttons_Switches_SMD:SW_SPST_B3U-1000P
- SW3: value SWITCH_INV -> BOOT0; footprint Buttons_Switches_SMD:SW_SPST_B3U-1100P-B -> Buttons_Switches_SMD:SW_SPST_B3U-3000P-B; moved to F.Cu
- U40: value CP2102N-24 -> CP2102N-A01-GQFN24
- moved SW1 5.85 mm to (31.8, -15.9)
- moved SW2 1.42 mm to (31.8, -15.9), turned to 315 degrees
- moved SW3 1.42 mm to (-15.9, 31.8), turned to 135 degrees
- moved C120 0.99 mm to (15.0, 15.9)
- moved D3 0.90 mm to (-24.1, -15.2)
- moved U2 0.54 mm to (13.7, 13.7)
- moved C121 0.46 mm to (-9.27, -10.2)
- moved C122 0.36 mm to (-7.62, 6.73)
- moved C117 0.28 mm to (-13.6, -12.7)
- moved C119 0.18 mm to (-10.2, 11.0)
- moved C123 0.13 mm to (11.6, 12.4)
- moved C4 0.10 mm to (6.35, 11.7), turned to 225 degrees
- turned C3 to 45 degrees
Connections:
- C3 pad 1: GND -> Net-(C3-Pad1)
- C3 pad 2: Net-(C3-Pad2) -> GND
- C4 pad 1: GND -> Net-(C4-Pad1)
- C4 pad 2: Net-(C4-Pad2) -> GND
- P1 pad 20: GND -> AVDD
- P2 pad 20: GND -> AVDD
- P3 pad 20: GND -> AVDD
- P4 pad 20: GND -> AVDD
- SW2 pad 1: GND -> Net-(R2-Pad2)
- SW3 pad 1: VCC_WIFI -> Net-(C126-Pad1)
- U37 pad 23: Net-(C3-Pad2) -> Net-(C3-Pad1)
- U37 pad 24: Net-(C4-Pad2) -> Net-(R1-Pad2)
- U5 pad 18: BOOT_WIFI -> Net-(C127-Pad1)
- U5 pad 3: VCC_WIFI -> Net-(C126-Pad1)
- Y2 pad 1: Net-(C4-Pad2) -> Net-(C4-Pad1)
- Y2 pad 2: Net-(C3-Pad2) -> Net-(C3-Pad1)
Routing:
- net AVDD: track 133.5 -> 208.5 mm, vias 17 -> 19
- net Net-(C127-Pad1): track 0.00 -> 26.4 mm, vias 0 -> 1
- net Net-(R2-Pad2): track 0.00 -> 25.4 mm, vias 0 -> 1
- net BOOT_WIFI: track 21.5 -> 0.00 mm, vias 1 -> 0
- net GND_ISO_UART: track 153.6 -> 173.2 mm, vias 3 -> 4
- net Net-(U37-Pad7): track 35.8 -> 16.8 mm
- net IOVDD: track 140.9 -> 155.8 mm
- net USART1_RX: track 12.8 -> 0.25 mm
- net NRST: track 67.6 -> 76.3 mm
- net Net-(C3-Pad2): track 8.63 -> 0.00 mm, vias 1 -> 0
- net Net-(C3-Pad1): track 0.00 -> 8.63 mm, vias 0 -> 1
- net Net-(C126-Pad1): track 0.00 -> 8.12 mm
- net Net-(C4-Pad2): track 7.22 -> 0.00 mm, vias 1 -> 0
- net Net-(R1-Pad2): track 0.00 -> 5.61 mm, vias 0 -> 1
- net VCC_WIFI: track 38.6 -> 44.0 mm
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Other:
- board size 70 x 70 mm -> 69.8 x 69.8 mm

Commit message: kicad
Parts:
- added C128: 100n, Capacitors_SMD:C_0402, B.Cu at (17.7, -16.4)
- added C129: 10n, Capacitors_SMD:C_0402, B.Cu at (16.8, -17.3)
- added C130: 100n, Capacitors_SMD:C_0402, B.Cu at (16.1, -21.5)
- added C132: 10u, Capacitors_SMD:C_0603, B.Cu at (-4.32, -18.2)
- added C133: 100n, Capacitors_SMD:C_0402, B.Cu at (-5.33, -18.3)
- added C134: 100n, Capacitors_SMD:C_0402, B.Cu at (4.06, -19.4)
- added C135: 22u, Capacitors_SMD:C_0805, B.Cu at (4.57, -16.8)
- added C136: 10u, Capacitors_SMD:C_0603, B.Cu at (-18.2, 4.32)
- added C137: 100n, Capacitors_SMD:C_0402, B.Cu at (-18.2, 5.33)
- added C138: 100n, Capacitors_SMD:C_0402, B.Cu at (-19.4, -4.06)
- added C139: 22u, Capacitors_SMD:C_0805, B.Cu at (-16.8, -4.57)
- added C140: 10u, Capacitors_SMD:C_0603, B.Cu at (4.32, 18.2)
- added C141: 100n, Capacitors_SMD:C_0402, B.Cu at (5.33, 18.0)
- added C142: 100n, Capacitors_SMD:C_0402, B.Cu at (-4.06, 19.3)
- added C143: 22u, Capacitors_SMD:C_0805, B.Cu at (-4.57, 16.8)
- added C144: 10u, Capacitors_SMD:C_0603, B.Cu at (18.0, -4.19)
- added C145: 100n, Capacitors_SMD:C_0402, B.Cu at (18.0, -5.21)
- added C146: 100n, Capacitors_SMD:C_0402, B.Cu at (19.4, 4.06)
- added C147: 22u, Capacitors_SMD:C_0805, B.Cu at (16.8, 4.45)
- added U26: TPD4E1B06, TO_SOT_Packages_SMD:SC-70-6, B.Cu at (25.4, 10.2)
- added U33: TPD4E1B06, TO_SOT_Packages_SMD:SC-70-6, B.Cu at (9.53, -25.4)
- added U38: TPD4E1B06, TO_SOT_Packages_SMD:SC-70-6, B.Cu at (-10.2, 25.4)
- added U4: TPD4E1B06, TO_SOT_Packages_SMD:SC-70-6, B.Cu at (-25.4, -10.2)
- C120, C123, U2: moved to B.Cu
- moved C120 28.1 mm to (-12.4, 9.65)
- moved C106 27.1 mm to (-7.37, 9.78), turned to 135 degrees
- moved U2 24.6 mm to (-10.7, 10.7), turned to 45 degrees
- moved C123 22.7 mm to (-10.7, 7.87)
- moved U10 2.54 mm to (0.00, 25.4)
- moved U11 2.54 mm to (-5.08, 25.4)
- moved U15 2.54 mm to (-25.4, 10.2)
- moved U16 2.54 mm to (-25.4, 5.08)
- moved U17 2.54 mm to (-25.4, 0.00)
- moved U18 2.54 mm to (-25.4, -5.08)
- moved U22 2.54 mm to (-10.2, -25.4)
- moved U23 2.54 mm to (-5.08, -25.4)
- moved U24 2.54 mm to (0.00, -25.4)
- moved U25 2.54 mm to (5.08, -25.4)
- moved U29 2.54 mm to (25.4, -10.2)
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Connections:
- P1 pad 1: Net-(P1-Pad1) -> REF
- P1 pad 2: Net-(P1-Pad1) -> REF
- P2 pad 1: Net-(P2-Pad1) -> REF
- P2 pad 2: Net-(P2-Pad1) -> REF
- P3 pad 1: Net-(P3-Pad1) -> REF
- P3 pad 2: Net-(P3-Pad1) -> REF
- P4 pad 1: Net-(P4-Pad1) -> REF
- P4 pad 2: Net-(P4-Pad1) -> REF
- U10 pad 1: /ADC4/AIN5+ -> /ADC4/AIN4+
- U10 pad 2: /ADC4/AIN5- -> /ADC4/AIN4-
- U10 pad 4: /ADC4/AIN4- -> /ADC4/AIN3-
- U10 pad 5: /ADC4/AIN4+ -> /ADC4/AIN3+
- U11 pad 1: /ADC4/AIN7+ -> /ADC4/AIN6+
- U11 pad 2: /ADC4/AIN7- -> /ADC4/AIN6-
- U11 pad 4: /ADC4/AIN6- -> /ADC4/AIN5-
- U11 pad 5: /ADC4/AIN6+ -> /ADC4/AIN5+
- U12 pad 11: Net-(U12-Pad11) -> GND
- U12 pad 12: Net-(U12-Pad12) -> GND
- U12 pad 20: Net-(U12-Pad20) -> GND
- U12 pad 8: Net-(U12-Pad8) -> VDD
- U15 pad 1: /ADC1/AIN1+ -> /ADC1/AIN0+
- U15 pad 2: /ADC1/AIN1- -> /ADC1/AIN0-
- U15 pad 4: /ADC1/AIN0- -> REF
- U15 pad 5: /ADC1/AIN0+ -> REF
- U16 pad 1: /ADC1/AIN3+ -> /ADC1/AIN2+
- U16 pad 2: /ADC1/AIN3- -> /ADC1/AIN2-
- U16 pad 4: /ADC1/AIN2- -> /ADC1/AIN1-
- U16 pad 5: /ADC1/AIN2+ -> /ADC1/AIN1+
- U17 pad 1: /ADC1/AIN5+ -> /ADC1/AIN4+
- U17 pad 2: /ADC1/AIN5- -> /ADC1/AIN4-
- U17 pad 4: /ADC1/AIN4- -> /ADC1/AIN3-
- U17 pad 5: /ADC1/AIN4+ -> /ADC1/AIN3+
- U18 pad 1: /ADC1/AIN7+ -> /ADC1/AIN6+
- U18 pad 2: /ADC1/AIN7- -> /ADC1/AIN6-
- U18 pad 4: /ADC1/AIN6- -> /ADC1/AIN5-
- U18 pad 5: /ADC1/AIN6+ -> /ADC1/AIN5+
- U22 pad 1: /ADC2/AIN1+ -> /ADC2/AIN0+
- U22 pad 2: /ADC2/AIN1- -> /ADC2/AIN0-
- U22 pad 4: /ADC2/AIN0- -> REF
- U22 pad 5: /ADC2/AIN0+ -> REF
- U23 pad 1: /ADC2/AIN3+ -> /ADC2/AIN2+
- U23 pad 2: /ADC2/AIN3- -> /ADC2/AIN2-
- U23 pad 4: /ADC2/AIN2- -> /ADC2/AIN1-
- U23 pad 5: /ADC2/AIN2+ -> /ADC2/AIN1+
- U24 pad 1: /ADC2/AIN5+ -> /ADC2/AIN4+
- U24 pad 2: /ADC2/AIN5- -> /ADC2/AIN4-
- U24 pad 4: /ADC2/AIN4- -> /ADC2/AIN3-
- U24 pad 5: /ADC2/AIN4+ -> /ADC2/AIN3+
- U25 pad 1: /ADC2/AIN7+ -> /ADC2/AIN6+
- U25 pad 2: /ADC2/AIN7- -> /ADC2/AIN6-
- U25 pad 4: /ADC2/AIN6- -> /ADC2/AIN5-
- U25 pad 5: /ADC2/AIN6+ -> /ADC2/AIN5+
- U29 pad 1: /ADC3/AIN1+ -> /ADC3/AIN0+
- U29 pad 2: /ADC3/AIN1- -> /ADC3/AIN0-
- U29 pad 4: /ADC3/AIN0- -> REF
- U29 pad 5: /ADC3/AIN0+ -> REF
- U30 pad 1: /ADC3/AIN3+ -> /ADC3/AIN2+
- U30 pad 2: /ADC3/AIN3- -> /ADC3/AIN2-
- U30 pad 4: /ADC3/AIN2- -> /ADC3/AIN1-
- U30 pad 5: /ADC3/AIN2+ -> /ADC3/AIN1+
- U31 pad 1: /ADC3/AIN5+ -> /ADC3/AIN4+
- U31 pad 2: /ADC3/AIN5- -> /ADC3/AIN4-
- U31 pad 4: /ADC3/AIN4- -> /ADC3/AIN3-
- U31 pad 5: /ADC3/AIN4+ -> /ADC3/AIN3+
- U32 pad 1: /ADC3/AIN7+ -> /ADC3/AIN6+
- U32 pad 2: /ADC3/AIN7- -> /ADC3/AIN6-
- U32 pad 4: /ADC3/AIN6- -> /ADC3/AIN5-
- U32 pad 5: /ADC3/AIN6+ -> /ADC3/AIN5+
- U37 pad 137: (no net) -> Net-(U37-Pad137)
- U37 pad 138: Net-(U37-Pad138) -> Net-(R2-Pad2)
- U43 pad 1: Net-(U43-Pad1) -> SDIO_D2
- U8 pad 1: /ADC4/AIN1+ -> /ADC4/AIN0+
- U8 pad 2: /ADC4/AIN1- -> /ADC4/AIN0-
- U8 pad 4: /ADC4/AIN0- -> REF
- U8 pad 5: /ADC4/AIN0+ -> REF
- U9 pad 1: /ADC4/AIN3+ -> /ADC4/AIN2+
- U9 pad 2: /ADC4/AIN3- -> /ADC4/AIN2-
- U9 pad 4: /ADC4/AIN2- -> /ADC4/AIN1-
- U9 pad 5: /ADC4/AIN2+ -> /ADC4/AIN1+
Routing:
- net GND: track 599.8 -> 1112.9 mm, vias 49 -> 48
- net REF: track 0.00 -> 289.5 mm
- net V+: track 76.7 -> 236.2 mm, vias 7 -> 8
- net AVDD: track 208.5 -> 335.0 mm
- net VDD: track 126.1 -> 210.3 mm, vias 5 -> 13
- net Net-(P1-Pad1): track 64.2 -> 0.00 mm
- net Net-(P2-Pad1): track 55.1 -> 0.00 mm
- net Net-(P3-Pad1): track 54.0 -> 0.00 mm
- net Net-(P4-Pad1): track 42.7 -> 0.00 mm
- net IOVDD: track 155.8 -> 123.6 mm
- net Net-(U37-Pad7): track 16.8 -> 0.00 mm, vias 1 -> 0
- net SDIO_D2: track 14.9 -> 28.7 mm
- net USART1_RX: track 0.25 -> 13.4 mm
- net Net-(R2-Pad2): track 25.4 -> 37.8 mm, vias 1 -> 2
- net Net-(U43-Pad1): track 12.3 -> 0.00 mm
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- added copper zone on In1.Cu, net AVDD
- added copper zone on In2.Cu, net GND
- added copper zone on In1.Cu, net IOVDD
- added copper zone on In1.Cu, net V+
- added copper zone on In1.Cu, net VDD
- removed copper zone on In2.Cu, net AVDD
- removed copper zone on In1.Cu, net GND
- removed copper zone on In2.Cu, net IOVDD
- removed copper zone on In2.Cu, net V+
- removed copper zone on In2.Cu, net VDD

Commit message: kicad
Parts:
- moved U33 0.63 mm to (10.2, -25.4)
- renumbered REF** to MH1, REF** to MH2, REF** to MH3, REF** to MH4
Routing:
- net VDD: track 210.3 -> 268.5 mm
- net GND: track 1112.9 -> 1117.8 mm, vias 48 -> 50
- net AVDD: track 335.0 -> 336.7 mm
- net REF: track 289.5 -> 290.1 mm, vias 0 -> 4
