File: KiCad/FreeEEG32.kicad_pcb (KiCad board)
At the start: 4 copper layers, 69.8 x 69.8 mm, 214 parts, among them P1 CONN_02X10, P11 CONN_01X03, P2 CONN_02X10, P3 CONN_02X10, P4 CONN_02X10, P6 CONN_02X03, P7 CONN_02X03, P8 USB_B, SW1 NRST, SW2 BOOT0, SW3 BOOT0, SW4 BOOT_WIFI, T1 da2303, U1 ADP7118AUJZ-3.3_TSOT, U10 TPD4E1B06, U11 TPD4E1B06, U12 MPU-6500, U13 AD7770, U14 ADR4525, U15 TPD4E1B06, U16 TPD4E1B06, U17 TPD4E1B06, U18 TPD4E1B06, U19 TLV73333PDBVT, U2 ADP7118AUJZ-3.3_TSOT, U20 AD7770, U21 ADR4525, U22 TPD4E1B06, U23 TPD4E1B06, U24 TPD4E1B06, U25 TPD4E1B06, U26 TPD4E1B06, U27 AD7770, U28 ADR4525, U29 TPD4E1B06, U3 8.192MHz, U30 TPD4E1B06, U31 TPD4E1B06, U32 TPD4E1B06, U33 TPD4E1B06, U34 AD7770, U35 ADUM1402BRWZ, U36 ISO7341c_spi, U37 STM32F427ZI_4side_short, U38 TPD4E1B06, U39 ADP7118AUJZ-3.3_TSOT, U4 TPD4E1B06, U40 CP2102N-A01-GQFN24, U43 473521001, U5 ESP-12F, U6 SN6505A, U7 ADR4525, U8 TPD4E1B06, U9 TPD4E1B06, Y2 8MHz

Commit message: kicad
Parts:
- added C131: CL2, Capacitors_SMD:C_0402, F.Cu at (7.62, 10.2)
- added J1: CONN_01X02, Socket_Strips:Socket_Strip_Straight_1x02, F.Cu at (27.9, -15.9)
- added Y1: 32768Hz, Crystals:Crystal_SMD_MicroCrystal_CC4V-T1A-2pin_5.0x1.9mm, F.Cu at (9.40, 9.40)
- C129: value 10n -> CL1; moved to F.Cu
- T1: footprint SMT_Power_Transformer:SMT Power Transformer -> da2303:da2303
- U1, U2, U39: value ADP7118AUJZ-3.3_TSOT -> ADP7118AUJZ-3.3
- U12: value MPU-6500 -> LSM6DS3; footprint Housings_DFN_QFN:QFN-24-1EP_4x4mm_Pitch0.5mm -> Housings_LGA_FreeEEG32:LGA-14L_2.5x3mm_Pitch0.5mm
- moved C129 25.1 mm to (9.27, 6.73), turned to 315 degrees
- moved C128 6.38 mm to (21.0, -21.8), turned to 45 degrees
- moved C130 5.74 mm to (21.8, -21.0), turned to 45 degrees
- moved R1 5.06 mm to (9.14, 12.2), turned to 45 degrees
- moved Y2 4.31 mm to (13.2, 13.2), turned to 45 degrees
- moved C125 1.63 mm to (30.5, -14.2)
- moved R2 1.63 mm to (30.5, -14.2)
- moved U6 0.90 mm to (-17.1, 26.0)
- moved C113 0.81 mm to (-18.8, 27.9)
- moved C107 0.72 mm to (-14.9, -9.53)
- moved C108 0.72 mm to (14.9, 9.53)
- moved SW1 0.45 mm to (32.1, -15.6)
- moved SW2 0.45 mm to (32.1, -15.6)
- moved SW3 0.45 mm to (-15.6, 32.1)
- moved SW4 0.45 mm to (-15.6, 32.1)
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Connections:
- C122 pad 1: AVDD -> IOVDD
- C123 pad 1: IOVDD -> AVDD
- C129 pad 1: GND -> Net-(C129-Pad1)
- C129 pad 2: Net-(C129-Pad2) -> GND
- C132 pad 2: V+ -> AVDD
- C133 pad 2: V+ -> AVDD
- C136 pad 2: V+ -> AVDD
- C137 pad 2: V+ -> AVDD
- C140 pad 2: V+ -> AVDD
- C141 pad 2: V+ -> AVDD
- C144 pad 2: V+ -> AVDD
- C145 pad 2: V+ -> AVDD
- P1 pad 1: REF -> AINREF
- P1 pad 2: REF -> /ADC4/VCM
- P2 pad 1: REF -> AINREF
- P2 pad 2: REF -> /ADC1/VCM
- P3 pad 1: REF -> AINREF
- P3 pad 2: REF -> /ADC2/VCM
- P4 pad 1: REF -> AINREF
- P4 pad 2: REF -> /ADC3/VCM
- U1 pad 4: AVDD -> IOVDD
- U1 pad 5: AVDD -> IOVDD
- U12 pad 1: Net-(U12-Pad1) -> SPI6_MISO
- U12 pad 10: Net-(C129-Pad2) -> Net-(U12-Pad10)
- U12 pad 11: GND -> Net-(U12-Pad11)
- U12 pad 12: GND -> SPI6_NSS
- U12 pad 13: VDD -> SPI6_SCK
- U12 pad 14: Net-(U12-Pad14) -> SPI6_MOSI
- U12 pad 2: Net-(U12-Pad2) -> GND
- U12 pad 3: Net-(U12-Pad3) -> GND
- U12 pad 5: Net-(U12-Pad5) -> VDD
- U12 pad 6: Net-(U12-Pad6) -> GND
- U12 pad 7: Net-(U12-Pad7) -> GND
- U12 pad 9: SPI6_MISO -> Net-(U12-Pad9)
- U14 pad 2: V+ -> AVDD
- U15 pad 4: REF -> AINREF
- U15 pad 5: REF -> /ADC1/VCM
- U2 pad 4: IOVDD -> AVDD
- U2 pad 5: IOVDD -> AVDD
- U21 pad 2: V+ -> AVDD
- U22 pad 4: REF -> AINREF
- U22 pad 5: REF -> /ADC2/VCM
- U28 pad 2: V+ -> AVDD
- U29 pad 4: REF -> AINREF
- U29 pad 5: REF -> /ADC3/VCM
- U37 pad 8: Net-(U37-Pad8) -> Net-(C129-Pad1)
- U7 pad 2: V+ -> AVDD
- U8 pad 4: REF -> AINREF
- U8 pad 5: REF -> /ADC4/VCM
Routing:
- net REF: track 290.1 -> 0.00 mm, vias 4 -> 0
- net AINREF: track 0.00 -> 207.4 mm, vias 0 -> 3
- net GND_ISO_UART: track 173.2 -> 108.0 mm, vias 4 -> 5
- net V+_ISO_UART: track 108.4 -> 68.8 mm, vias 1 -> 3
- net AVDD: track 336.7 -> 370.2 mm, vias 19 -> 17
- net /ADC2/VCM: track 7.99 -> 29.7 mm
- net /ADC1/VCM: track 7.99 -> 29.6 mm
- net /ADC3/VCM: track 7.99 -> 29.3 mm
- net /ADC4/VCM: track 8.16 -> 29.3 mm
- net /ADC3/REF1+: track 46.7 -> 67.2 mm
- net /ADC1/REF1+: track 48.0 -> 67.8 mm
- net V+: track 236.2 -> 216.6 mm, vias 8 -> 4
- net /ADC4/REF1+: track 49.1 -> 68.4 mm
- net Net-(C131-Pad1): track 0.00 -> 16.3 mm, vias 0 -> 1
- net Net-(C129-Pad1): track 0.00 -> 13.9 mm, vias 0 -> 1
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- added copper zone on In2.Cu, net GND_ISO_SPI
- added copper zone on In2.Cu, net GND_ISO_UART
- added copper zone on In1.Cu, net V+_ISO_SPI
- added copper zone on In1.Cu, net V+_ISO_UART
Other:
- board text added: "V+_ISO"

Commit message: kicad
Routing:
- net GND: track 1115.3 -> 1088.1 mm, vias 64 -> 80
- net AVDD: track 370.2 -> 358.5 mm
Other:
- board text added: "FreeEEG32 alpha"
- board text added: "neuroidss.com"
