File: KiCad/FreeEEG32.sch (KiCad schematic (older format))
At the start: 30 parts, among them P11 CONN_01X03, SW1 NRST, U1 ADP7118AUJZ-3.3_TSOT, U2 ADP7118AUJZ-3.3_TSOT, U3 8.192MHz, U37 STM32F427ZI_4side_short, U39 ADP7118AUJZ-3.3_TSOT, U4 STM32F427ZI_4side, U43 473521001, Y1 32.768kHz, Y2 8MHz

Commit message: kicad
Parts:
- added C118: 100n, Capacitors_SMD:C_0402, symbol C_Small
- Y2: footprint Crystals:Crystal_SMD_5032-4pin_5.0x3.2mm -> Crystals:Crystal_SMD_5032_4Pads
Connections:
- wire segments 292 -> 302
Other:
- moved on the sheet: C1, C10, C100, C101, C102, C103, C104, C105, C106, C11, C2, C3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

Commit message: kicad & restructure catalogs
Changed lines of the file:
@@
 Text GLabel 8250 1150 1    60   Input ~ 0
 AD2_START
-Text GLabel 7550 1150 1    60   Input ~ 0
+Text GLabel 7950 1150 1    60   Input ~ 0
 AD2_RESET
 Text GLabel 11900 2250 2    60   Input ~ 0
@@
 	11850 2250 11900 2250
 Wire Wire Line
-	7550 1200 7550 1150
+	7950 1200 7950 1150
 Wire Wire Line
 	8250 1200 8250 1150

Commit message: kicad
Connections:
- wire segments 302 -> 300
Changed lines of the file:
@@
 	1    0    0    -1
 $EndComp
-Text GLabel 9650 8450 3    60   Input ~ 0
+Text GLabel 9050 5250 3    60   Input ~ 0
 I2C2_SDA
-Text GLabel 9550 8450 3    60   Input ~ 0
+Text GLabel 8950 5250 3    60   Input ~ 0
 I2C2_SCL
 $Comp
@@
 	10900 2850 10950 2850
 Wire Wire Line
-	9300 5500 9300 5600
-Wire Wire Line
-	9100 5500 9100 5600
-Wire Wire Line
-	9100 5550 9100 5250
-Connection ~ 9100 5550
-Connection ~ 9300 5550
+	9100 5250 9100 5600
 Wire Wire Line
 	9100 5250 9150 5250
@@
 	10900 1550 10950 1550
 Wire Wire Line
-	9300 5550 9300 5450
+	9300 5450 9300 5600
 Wire Wire Line
 	9300 5450 9150 5450
@@
 	8500 6250 8550 6250
 Wire Wire Line
-	9550 8450 9550 8400
-Wire Wire Line
-	9650 8450 9650 8400
+	8950 5250 8950 5200
+Wire Wire Line
+	9050 5250 9050 5200
 $Sheet
 S 600  4450 1100 900
@@
 Wire Wire Line
 	10900 3950 10950 3950
+Connection ~ 9300 5550
+Connection ~ 9100 5550
 $EndSCHEMATC

Commit message: kicad
Parts:
- removed R1: REXT, Resistors_SMD:R_0402, symbol R_Small
- removed Y1: 32.768kHz, Crystals:Crystal_SMD_0603_2Pads_obsolete, symbol Crystal_Small
- added C116: 1u, Capacitors_SMD:C_0402, symbol C_Small
- added C117, C119, C120, C121, C122, C123, C124: 2.2u, Capacitors_SMD:C_0603, symbol C_Small
- added SW2: SWITCH_INV, Buttons_Switches_SMD:SW_SPST_B3U-1100P-B, symbol SWITCH_INV
- added U12: MPU-6500, Housings_DFN_QFN:QFN-24-1EP_4x4mm_Pitch0.5mm, symbol MPU-6500
- C1: value CL1 -> 100n
- C102: footprint Capacitors_SMD:C_0402 -> Capacitors_SMD:C_0603; manf# (none) -> GRM188R60J225KE19D
- C106: footprint Capacitors_SMD:C_0402 -> Capacitors_SMD:C_0603; manf# (none) -> GRM188R60J475KE19D
- C2: value CL2 -> 1u
Connections:
- net AVDD: now also U1.4 (SENSE/ADJ), C122.1
- net BOOT0: now also SW2.3
- net GND: now also C7.2, U37.31 (VSSA), C116.1, C117.2, C119.2, C120.2, C121.2, C122.2, C123.2, C124.2, SW2.1, U12.18 (GND); no longer C7.1, U37.30 (VDD)
- net IOVDD: now also U2.4 (SENSE/ADJ), C123.1
- net NRST: now also U37.27 (PC1\ADC123_IN11); no longer C5.2, U37.25 (NRST)
- net SDIO_D2: no longer U43.1 (DATA2)
- net SDIO_DETECT: now also U37.97 (PC7|I2S3_MCK/SDIO_D7/USART6_RX); no longer U37.100 (PA8|MCO1/I2C3_SCL)
- net SPI6_MISO: now also U12.9 (AD0/SDO)
- net SPI6_MOSI: now also U12.24 (SDA/SDI)
- net SPI6_NSS: now also U12.22 (nCS)
- net SPI6_SCK: now also U12.23 (SCL/SCLK)
- net V+: now also C117.1, C119.1, C120.1
- net VDD: now also C1.2, C103.2, C2.2, C5.2, C7.1, U37.30 (VDD), U37.32 (VREF+), U37.33 (VDDA), U37.6 (VBAT), U37.72 (VDD), U39.4 (SENSE/ADJ), C116.2, C121.1, SW2.2, U12.13 (VDD); no longer C102.1, C7.2, U37.31 (VSSA), U37.71 (VCAP_1)
- net at U37.9 (PC15/OSC32_OUT): no longer C2.2
- net at U37.8 (PC14/OSC32_IN): no longer C1.2
- net at U37.106 (VCAP_2): now also C124.1
- new net: C102.1, U37.71 (VCAP_1)
Other:
- moved on the sheet: C10, C100, C101, C102, C103, C104, C105, C106, C11, C118, C6, C7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

Commit message: kicad
Parts:
- removed U4: STM32F427ZI_4side, symbol STM32F427ZI_4side
- C1, C10, C100, C101, C103, C104, C105, C11, C118, C5, C6, C7, C8, C9: manf# (none) -> MC0402B104K160CT
- C116, C2: manf# (none) -> GRM155R60J105KE19D
- C117, C119, C120, C121, C122, C123: manf# (none) -> GRM188R60J225KE19D
- P11: manf# (none) -> PBS-3
- U3: manf# 7W-8.192MBC-T -> 7W-8.192MBA-T
- U43: manf# (none) -> 473521001

Commit message: kicad
Connections:
- net NRST: now also U37.25 (NRST); no longer U37.27 (PC1\ADC123_IN11)
Changed lines of the file:
@@
 	3300 4450 3250 4450
-Wire Wire Line
-	3650 4050 4250 4050
 Wire Wire Line
 	4200 3750 4250 3750
@@
 Wire Wire Line
 	4850 900  4800 900
+Wire Wire Line
+	4150 4050 4150 3850
+Wire Wire Line
+	4150 3850 4250 3850
+Wire Wire Line
+	4150 4050 3650 4050
 $EndSCHEMATC

Commit message: kicad
Parts:
- removed SW2: SWITCH_INV, Buttons_Switches_SMD:SW_SPST_B3U-1100P-B, symbol SWITCH_INV
- added C125: 100n, Capacitors_SMD:C_0402, symbol C_Small
- added R1: R_EXT, Resistors_SMD:R_0402, symbol R_Small
- added R2, R3: 47k, Resistors_SMD:R_0402, symbol R_Small
- added SW2: BOOT0, Buttons_Switches_SMD:SW_SPST_B3U-1000P, symbol SW_PUSH_SMALL
- SW1: footprint Buttons_Switches_SMD:SW_SPST_B3U-1000P-B -> Buttons_Switches_SMD:SW_SPST_B3U-3000P-B; manf# (none) -> B3U3000PMB
Connections:
- net BOOT0 is gone; now on an unnamed net: U37.138 (PB7|I2C1_SDA/FSMC_NL)
- net GND: now also C3.2, C4.2, C125.1, R2.1, R3.2; no longer C3.1, C4.1
- net NRST: now also C125.2
- net VDD: now also SW2.2
- net at U37.23 (PH0/OSC_IN), Y2.2: now also C3.1; no longer C3.2
- net at U37.138 (PB7|I2C1_SDA/FSMC_NL): now also R2.2, SW2.1
- net at U37.48 (PB2/BOOT1): now also R3.1
- new net: C4.1, R1.1, Y2.1
- new net: R1.2, U37.24 (PH1/OSC_OUT)
Other:
- moved on the sheet: C3, C4, P11, SW1, Y2
Changed lines of the file:
@@
 L Crystal_Small Y2
 U 1 1 5841A270
-P 4050 3700
-F 0 "Y2" H 4050 3800 50  0000 C CNN
-F 1 "8MHz" H 4050 3600 50  0000 C CNN
-F 2 "Crystals:Crystal_SMD_5032_4Pads" H 4050 3700 50  0001 C CNN
-F 3 "" H 4050 3700 50  0000 C CNN
-F 4 "KX-9A 8.0 MHz" H 4050 3700 60  0000 C CNN "manf#"
-	1    4050 3700
+P 3900 3700
+F 0 "Y2" H 3900 3800 50  0000 C CNN
+F 1 "8MHz" H 3900 3600 50  0000 C CNN
+F 2 "Crystals:Crystal_SMD_5032_4Pads" H 3900 3700 50  0001 C CNN
+F 3 "" H 3900 3700 50  0000 C CNN
+F 4 "KX-9A 8.0 MHz" H 3900 3700 60  0001 C CNN "manf#"
+	1    3900 3700
 	0    -1   -1   0
 $EndComp
@@
 L C_Small C3
 U 1 1 5841A27C
-P 3650 3650
-F 0 "C3" H 3660 3720 50  0000 L CNN
-F 1 "CL1" H 3660 3570 50  0000 L CNN
-F 2 "Capacitors_SMD:C_0402" H 3650 3650 50  0001 C CNN
-F 3 "" H 3650 3650 50  0000 C CNN
-	1    3650 3650
-	0    -1   -1   0
+P 3700 3600
+F 0 "C3" H 3710 3670 50  0000 L CNN
+F 1 "CL1" H 3710 3520 50  0000 L CNN
+F 2 "Capacitors_SMD:C_0402" H 3700 3600 50  0001 C CNN
+F 3 "" H 3700 3600 50  0000 C CNN
+	1    3700 3600
+	0    1    1    0
 $EndComp
 $Comp
 L C_Small C4
 U 1 1 5841A28E
-P 3800 3750
-F 0 "C4" H 3810 3820 50  0000 L CNN
-F 1 "CL2" H 3810 3670 50  0000 L CNN
-F 2 "Capacitors_SMD:C_0402" H 3800 3750 50  0001 C CNN
-F 3 "" H 3800 3750 50  0000 C CNN
-	1    3800 3750
-	0    -1   -1   0
-$EndComp
-Text GLabel 3650 3900 0    60   Input ~ 0
+P 3700 3800
+F 0 "C4" H 3710 3870 50  0000 L CNN
+F 1 "CL2" H 3710 3720 50  0000 L CNN
+F 2 "Capacitors_SMD:C_0402" H 3700 3800 50  0001 C CNN
+F 3 "" H 3700 3800 50  0000 C CNN
+	1    3700 3800
+	0    1    1    0
+$EndComp
+Text GLabel 3500 3900 0    60   Input ~ 0
 VSS
 $Comp
@@
 L SW_PUSH_SMALL SW1
 U 1 1 5841A2AD
-P 4000 3950
-F 0 "SW1" H 4150 4060 50  0000 C CNN
-F 1 "NRST" H 4000 3871 50  0000 C CNN
-F 2 "Buttons_Switches_SMD:SW_SPST_B3U-1000P-B" H 4000 3950 50  0001 C CNN
-F 3 "" H 4000 3950 50  0000 C CNN
-	1    4000 3950
+P 3850 4000
+F 0 "SW1" H 4000 4110 50  0000 C CNN
+F 1 "NRST" H 3850 3921 50  0000 C CNN
+F 2 "Buttons_Switches_SMD:SW_SPST_B3U-3000P-B" H 3850 4000 50  0001 C CNN
+F 3 "" H 3850 4000 50  0000 C CNN
+F 4 "B3U3000PMB" H 3850 4000 60  0001 C CNN "manf#"
+	1    3850 4000
 	-1   0    0    1
 $EndComp
-Text GLabel 3650 4050 0    60   Input ~ 0
+Text GLabel 3650 4100 0    60   Input ~ 0
 NRST
 Text GLabel 10300 1750 2    60   Input ~ 0
@@
 Text GLabel 6600 1150 1    60   Input ~ 0
 SPI3_SCK
-Text GLabel 6100 1150 1    60   Input ~ 0
-BOOT0
 Text GLabel 4200 1450 0    60   Input ~ 0
 SPI4_SCK
@@
 L CONN_01X03 P11
 U 1 1 58BA2E74
-P 6700 7250
-F 0 "P11" H 6700 7450 50  0000 C CNN
-F 1 "CONN_01X03" V 6800 7250 50  0000 C CNN
-F 2 "Socket_Strips:Socket_Strip_Straight_1x03" H 6700 7250 50  0001 C CNN
-F 3 "" H 6700 7250 50  0000 C CNN
-F 4 "PBS-3" H 6700 7250 60  0001 C CNN "manf#"
-	1    6700 7250
+P 4600 1100
+F 0 "P11" H 4600 1300 50  0000 C CNN
+F 1 "CONN_01X03" V 4700 1100 50  0000 C CNN
+F 2 "Socket_Strips:Socket_Strip_Straight_1x03" H 4600 1100 50  0001 C CNN
+F 3 "" H 4600 1100 50  0000 C CNN
+F 4 "PBS-3" H 4600 1100 60  0001 C CNN "manf#"
+	1    4600 1100
 	0    1    1    0
 $EndComp
-Text GLabel 6800 7000 1    60   Input ~ 0
+Text GLabel 4700 850  1    60   Input ~ 0
 SWCLK
-Text GLabel 6700 7000 1    60   Input ~ 0
+Text GLabel 4600 850  1    60   Input ~ 0
 SWDIO
-Text GLabel 6600 7000 1    60   Input ~ 0
+Text GLabel 4500 850  1    60   Input ~ 0
 NRST
 Text GLabel 4200 4850 0    60   Input ~ 0
@@
 	4200 4950 4250 4950
 Wire Wire Line
-	3900 3800 4200 3800
+	3800 3800 4000 3800
 Wire Wire Line
 	4200 3800 4200 3750
-Connection ~ 4050 3600
-Connection ~ 4050 3800
-Wire Wire Line
-	3550 3750 3700 3750
-Wire Wire Line
-	3700 3750 3700 3900
-Connection ~ 3550 3650
-Connection ~ 3700 3750
-Wire Wire Line
-	3900 3600 4200 3600
+Connection ~ 3900 3600
+Connection ~ 3900 3800
+Wire Wire Line
+	3800 3600 4200 3600
 Connection ~ 4000 3100
 Connection ~ 4000 2900
@@
 Wire Wire Line
 	3850 2950 3900 2950
-Connection ~ 4100 4050
-Wire Wire Line
-	3700 3850 3900 3850
-Connection ~ 3700 3850
-Wire Wire Line
-	3700 3900 3650 3900
+Connection ~ 3950 4100
+Wire Wire Line
+	3500 3900 4050 3900
 Wire Wire Line
 	10250 1750 10300 1750
@@
 	6400 1200 6400 1150
 Wire Wire Line
-	6100 1150 6100 1200
-Wire Wire Line
 	4250 1850 4200 1850
 Wire Wire Line
@@
 	10250 1850 10300 1850
 Wire Wire Line
-	6800 7000 6800 7050
-Wire Wire Line
-	6700 7000 6700 7050
-Wire Wire Line
-	6600 7000 6600 7050
+	4700 850  4700 900
+Wire Wire Line
+	4600 850  4600 900
+Wire Wire Line
+	4500 850  4500 900
 Wire Wire Line
 	4250 4750 4200 4750
@@
 Wire Wire Line
 	4200 3600 4200 3650
-Wire Wire Line
-	3900 3600 3900 3650
-Wire Wire Line
-	3900 3650 3750 3650
-Wire Wire Line
-	3550 3750 3550 3650
-Wire Wire Line
-	3900 3800 3900 3750
 Wire Wire Line
 	5600 6400 5600 6600
@@
 Wire Wire Line
 	4200 1950 4250 1950
-Text GLabel 4850 700  2    60   Input ~ 0
-VSS
-Text GLabel 3750 800  0    60   Input ~ 0
-VDD
-Wire Wire Line
-	3800 800  3750 800
-Wire Wire Line
-	4800 700  4850 700
-Text GLabel 4850 900  2    60   Input ~ 0
-BOOT0
-$Comp
-L SWITCH_INV SW2
-U 1 1 58E042BC
-P 4300 800
-F 0 "SW2" H 4100 950 50  0000 C CNN
-F 1 "SWITCH_INV" H 4150 650 50  0000 C CNN
-F 2 "Buttons_Switches_SMD:SW_SPST_B3U-1100P-B" H 4300 800 50  0001 C CNN
-F 3 "" H 4300 800 50  0000 C CNN
-	1    4300 800
-	1    0    0    -1
-$EndComp
-Wire Wire Line
-	4850 900  4800 900
-Wire Wire Line
-	4150 4050 4150 3850
+Wire Wire Line
+	4150 4100 4150 3850
 Wire Wire Line
 	4150 3850 4250 3850
 Wire Wire Line
-	4150 4050 3650 4050
+	3650 4100 4150 4100
 $Comp
 L MPU-6500 U12
@@
 	1    0    0    -1
 $EndComp
+Text GLabel 6600 5500 3    60   Input ~ 0
+VSS
+Wire Wire Line
+	6600 5200 6600 5250
+$Comp
+L C_Small C125
+U 1 1 58E42B84
+P 4050 4000
+F 0 "C125" H 4060 4070 50  0000 L CNN
+F 1 "100n" H 4060 3920 50  0000 L CNN
+F 2 "Capacitors_SMD:C_0402" H 4050 4000 50  0001 C CNN
+F 3 "" H 4050 4000 50  0000 C CNN
+F 4 "MC0402B104K160CT" H 4050 4000 60  0001 C CNN "manf#"
+	1    4050 4000
+	1    0    0    -1
+$EndComp
+Wire Wire Line
+	3950 4100 4050 4100
+Connection ~ 4050 4100
+Connection ~ 3750 3900
+$Comp
+L R_Small R1
+U 1 1 58E45491
+P 4100 3800
+F 0 "R1" H 4130 3820 50  0000 L CNN
+F 1 "R_EXT" H 4130 3760 50  0000 L CNN
+F 2 "Resistors_SMD:R_0402" H 4100 3800 50  0001 C CNN
+F 3 "" H 4100 3800 50  0000 C CNN
+	1    4100 3800
+	0    -1   -1   0
+$EndComp
+Wire Wire Line
+	3600 3600 3550 3600
+Wire Wire Line
+	3550 3600 3550 3900
+Wire Wire Line
+	3600 3800 3550 3800
+Connection ~ 3550 3800
+Connection ~ 3550 3900
+$Comp
+L R_Small R3
+U 1 1 58E49D48
+P 6600 5350
+F 0 "R3" H 6630 5370 50  0000 L CNN
+F 1 "47k" H 6630 5310 50  0000 L CNN
+F 2 "Resistors_SMD:R_0402" H 6600 5350 50  0001 C CNN
+F 3 "" H 6600 5350 50  0000 C CNN
+F 4 "RC0402FR-0747KL" H 6600 5350 60  0001 C CNN "manf#"
+	1    6600 5350
+	1    0    0    -1
+$EndComp
+Wire Wire Line
+	6600 5500 6600 5450
+$Comp
+L R_Small R2
+U 1 1 58E4B6DE
+P 6150 1050
+F 0 "R2" H 6180 1070 50  0000 L CNN
+F 1 "47k" H 6180 1010 50  0000 L CNN
+F 2 "Resistors_SMD:R_0402" H 6150 1050 50  0001 C CNN
+F 3 "" H 6150 1050 50  0000 C CNN
+F 4 "RC0402FR-0747KL" H 6150 1050 60  0001 C CNN "manf#"
+	1    6150 1050
+	1    0    0    -1
+$EndComp
+Text GLabel 6150 900  1    60   Input ~ 0
+VSS
+Wire Wire Line
+	6150 950  6150 900
+$Comp
+L SW_PUSH_SMALL SW2
+U 1 1 58E4FE38
+P 6000 1050
+F 0 "SW2" H 6150 1160 50  0000 C CNN
+F 1 "BOOT0" H 6000 971 50  0000 C CNN
+F 2 "Buttons_Switches_SMD:SW_SPST_B3U-1000P" H 6000 1050 50  0001 C CNN
+F 3 "" H 6000 1050 50  0000 C CNN
+F 4 "B3U1000P" H 6000 1050 60  0001 C CNN "manf#"
+	1    6000 1050
+	-1   0    0    1
+$EndComp
+Text GLabel 5900 900  1    60   Input ~ 0
+VDD
+Wire Wire Line
+	6100 1200 6100 1150
+Wire Wire Line
+	6100 1150 6150 1150
+Wire Wire Line
+	5900 950  5900 900
 $EndSCHEMATC
