File: KiCad/ADC.sch (KiCad schematic (older format))
At the start: 29 parts, among them P1 CONN_02X10, U10 TPD4E1B06, U11 TPD4E1B06, U12 TPD4E1B06, U13 AD7770, U7 ADR4525, U8 TPD4E1B06, U9 TPD4E1B06

Commit message: kicad
Connections:
- net CONVST_SAR is gone; now on net GND: U13.17 (CONVST_SAR)
Changed lines of the file:
@@
 $Descr A4 11693 8268
 encoding utf-8
-Sheet 5 6
+Sheet 4 6
 Title ""
 Date ""
@@
 AR Path="/58B5D98C/58B4BBD1" Ref="C61"  Part="1"
 AR Path="/58B5EE77/58B4BBD1" Ref="C82"  Part="1"
-F 0 "C61" H 5510 3970 50  0000 L CNN
+F 0 "C15" H 5510 3970 50  0000 L CNN
 F 1 "1u" H 5510 3820 50  0000 L CNN
 F 2 "Capacitors_SMD:C_0402" H 5500 3900 50  0001 C CNN
@@
 AR Path="/58B5D98C/58B4BBD8" Ref="C65"  Part="1"
 AR Path="/58B5EE77/58B4BBD8" Ref="C86"  Part="1"
-F 0 "C65" H 5760 3970 50  0000 L CNN
+F 0 "C19" H 5760 3970 50  0000 L CNN
 F 1 "100n" H 5760 3820 50  0000 L CNN
 F 2 "Capacitors_SMD:C_0402" H 5750 3900 50  0001 C CNN
@@
 AR Path="/58B5D98C/58B4BBDF" Ref="C64"  Part="1"
 AR Path="/58B5EE77/58B4BBDF" Ref="C85"  Part="1"
-F 0 "C64" H 5760 3670 50  0000 L CNN
+F 0 "C18" H 5760 3670 50  0000 L CNN
 F 1 "100n" H 5760 3520 50  0000 L CNN
 F 2 "Capacitors_SMD:C_0402" H 5750 3600 50  0001 C CNN
@@
 AR Path="/58B5D98C/58B4BBE6" Ref="C60"  Part="1"
 AR Path="/58B5EE77/58B4BBE6" Ref="C81"  Part="1"
-F 0 "C60" H 5510 3670 50  0000 L CNN
+F 0 "C14" H 5510 3670 50  0000 L CNN
 F 1 "1u" H 5510 3520 50  0000 L CNN
 F 2 "Capacitors_SMD:C_0402" H 5500 3600 50  0001 C CNN
@@
 AR Path="/58B5D98C/58B4BBED" Ref="C63"  Part="1"
 AR Path="/58B5EE77/58B4BBED" Ref="C84"  Part="1"
-F 0 "C63" H 5760 2270 50  0000 L CNN
+F 0 "C17" H 5760 2270 50  0000 L CNN
 F 1 "100n" H 5760 2120 50  0000 L CNN
 F 2 "Capacitors_SMD:C_0402" H 5750 2200 50  0001 C CNN
@@
 AR Path="/58B5D98C/58B4BBF4" Ref="C59"  Part="1"
 AR Path="/58B5EE77/58B4BBF4" Ref="C80"  Part="1"
-F 0 "C59" H 5510 2270 50  0000 L CNN
+F 0 "C13" H 5510 2270 50  0000 L CNN
 F 1 "1u" H 5510 2120 50  0000 L CNN
 F 2 "Capacitors_SMD:C_0402" H 5500 2200 50  0001 C CNN
@@
 AR Path="/58B5D98C/58B4BBFB" Ref="C62"  Part="1"
 AR Path="/58B5EE77/58B4BBFB" Ref="C83"  Part="1"
-F 0 "C62" H 5760 1970 50  0000 L CNN
+F 0 "C16" H 5760 1970 50  0000 L CNN
 F 1 "100n" H 5760 1820 50  0000 L CNN
 F 2 "Capacitors_SMD:C_0402" H 5750 1900 50  0001 C CNN
@@
 AR Path="/58B5D98C/58B4BC02" Ref="C58"  Part="1"
 AR Path="/58B5EE77/58B4BC02" Ref="C79"  Part="1"
-F 0 "C58" H 5510 1970 50  0000 L CNN
+F 0 "C12" H 5510 1970 50  0000 L CNN
 F 1 "1u" H 5510 1820 50  0000 L CNN
 F 2 "Capacitors_SMD:C_0402" H 5500 1900 50  0001 C CNN
@@
 AR Path="/58B5D98C/58B4BC09" Ref="C66"  Part="1"
 AR Path="/58B5EE77/58B4BC09" Ref="C87"  Part="1"
-F 0 "C66" H 8560 3570 50  0000 L CNN
+F 0 "C20" H 8560 3570 50  0000 L CNN
 F 1 "100n" H 8560 3420 50  0000 L CNN
 F 2 "Capacitors_SMD:C_0402" H 8550 3500 50  0001 C CNN
@@
 AR Path="/58B5D98C/58B4BC10" Ref="C73"  Part="1"
 AR Path="/58B5EE77/58B4BC10" Ref="C94"  Part="1"
-F 0 "C73" H 8810 3570 50  0000 L CNN
+F 0 "C29" H 8810 3570 50  0000 L CNN
 F 1 "1u" H 8810 3420 50  0000 L CNN
 F 2 "Capacitors_SMD:C_0402" H 8800 3500 50  0001 C CNN
@@
 AR Path="/58B5D98C/58B4BC17" Ref="C74"  Part="1"
 AR Path="/58B5EE77/58B4BC17" Ref="C95"  Part="1"
-F 0 "C74" H 8810 3870 50  0000 L CNN
+F 0 "C30" H 8810 3870 50  0000 L CNN
 F 1 "1u" H 8810 3720 50  0000 L CNN
 F 2 "Capacitors_SMD:C_0402" H 8800 3800 50  0001 C CNN
@@
 AR Path="/58B5D98C/58B4BC1E" Ref="C67"  Part="1"
 AR Path="/58B5EE77/58B4BC1E" Ref="C88"  Part="1"
-F 0 "C67" H 8560 3870 50  0000 L CNN
+F 0 "C21" H 8560 3870 50  0000 L CNN
 F 1 "100n" H 8560 3720 50  0000 L CNN
 F 2 "Capacitors_SMD:C_0402" H 8550 3800 50  0001 C CNN
@@
 AR Path="/58B5D98C/58B4BC25" Ref="C78"  Part="1"
 AR Path="/58B5EE77/58B4BC25" Ref="C99"  Part="1"
-F 0 "C78" H 8910 3070 50  0000 L CNN
+F 0 "C34" H 8910 3070 50  0000 L CNN
 F 1 "100n" H 8910 2920 50  0000 L CNN
 F 2 "Capacitors_SMD:C_0402" H 8900 3000 50  0001 C CNN
@@
 AR Path="/58B5D98C/58B4BC2C" Ref="C68"  Part="1"
 AR Path="/58B5EE77/58B4BC2C" Ref="C89"  Part="1"
-F 0 "C68" H 8310 2920 50  0000 L CNN
+F 0 "C22" H 8310 2920 50  0000 L CNN
 F 1 "100n" H 8310 2770 50  0000 L CNN
 F 2 "Capacitors_SMD:C_0402" H 8300 2850 50  0001 C CNN
@@
 AR Path="/58B5D98C/58B4BC33" Ref="C71"  Part="1"
 AR Path="/58B5EE77/58B4BC33" Ref="C92"  Part="1"
-F 0 "C71" H 8660 2870 50  0000 L CNN
+F 0 "C27" H 8660 2870 50  0000 L CNN
 F 1 "100n" H 8660 2720 50  0000 L CNN
 F 2 "Capacitors_SMD:C_0402" H 8650 2800 50  0001 C CNN
@@
 AR Path="/58B5D98C/58B4BC3A" Ref="C70"  Part="1"
 AR Path="/58B5EE77/58B4BC3A" Ref="C91"  Part="1"
-F 0 "C70" H 8660 2070 50  0000 L CNN
+F 0 "C26" H 8660 2070 50  0000 L CNN
 F 1 "100n" H 8660 1920 50  0000 L CNN
 F 2 "Capacitors_SMD:C_0402" H 8650 2000 50  0001 C CNN
@@
 AR Path="/58B5D98C/58B4BC41" Ref="C72"  Part="1"
 AR Path="/58B5EE77/58B4BC41" Ref="C93"  Part="1"
-F 0 "C72" H 8310 2020 50  0000 L CNN
+F 0 "C28" H 8310 2020 50  0000 L CNN
 F 1 "100n" H 8310 1870 50  0000 L CNN
 F 2 "Capacitors_SMD:C_0402" H 8300 1950 50  0001 C CNN
@@
 AR Path="/58B5D98C/58B4BC48" Ref="C69"  Part="1"
 AR Path="/58B5EE77/58B4BC48" Ref="C90"  Part="1"
-F 0 "C69" H 8660 1770 50  0000 L CNN
+F 0 "C23" H 8660 1770 50  0000 L CNN
 F 1 "100n" H 8660 1620 50  0000 L CNN
 F 2 "Capacitors_SMD:C_0402" H 8650 1700 50  0001 C CNN
@@
 AR Path="/58B5D98C/58B4BC4F" Ref="C77"  Part="1"
 AR Path="/58B5EE77/58B4BC4F" Ref="C98"  Part="1"
-F 0 "C77" H 8910 2870 50  0000 L CNN
+F 0 "C33" H 8910 2870 50  0000 L CNN
 F 1 "1u" H 8910 2720 50  0000 L CNN
 F 2 "Capacitors_SMD:C_0402" H 8900 2800 50  0001 C CNN
@@
 AR Path="/58B5D98C/58B4BC56" Ref="C76"  Part="1"
 AR Path="/58B5EE77/58B4BC56" Ref="C97"  Part="1"
-F 0 "C76" H 8910 2070 50  0000 L CNN
+F 0 "C32" H 8910 2070 50  0000 L CNN
 F 1 "1u" H 8910 1920 50  0000 L CNN
 F 2 "Capacitors_SMD:C_0402" H 8900 2000 50  0001 C CNN
@@
 AR Path="/58B5D98C/58B4BC5D" Ref="C75"  Part="1"
 AR Path="/58B5EE77/58B4BC5D" Ref="C96"  Part="1"
-F 0 "C75" H 8910 1770 50  0000 L CNN
+F 0 "C31" H 8910 1770 50  0000 L CNN
 F 1 "1u" H 8910 1620 50  0000 L CNN
 F 2 "Capacitors_SMD:C_0402" H 8900 1700 50  0001 C CNN
@@
 AR Path="/58B5D98C/58B4BD09" Ref="U27"  Part="1"
 AR Path="/58B5EE77/58B4BD09" Ref="U34"  Part="1"
-F 0 "U27" H 7150 3100 60  0000 C CNN
+F 0 "U13" H 7150 3100 60  0000 C CNN
 F 1 "AD7770" H 7150 3000 60  0000 C CNN
 F 2 "Housings_DFN_QFN:QFN-64-1EP_9x9mm_Pitch0.5mm" H 7150 3050 60  0001 C CNN
@@
 AR Path="/58B5D98C/58B4BD10" Ref="U21"  Part="1"
 AR Path="/58B5EE77/58B4BD10" Ref="U28"  Part="1"
-F 0 "U21" H 2400 3700 60  0000 C CNN
+F 0 "U7" H 2400 3700 60  0000 C CNN
 F 1 "ADR4525" H 2400 4200 60  0000 C CNN
 F 2 "Housings_SOIC:SOIC-8_3.9x4.9mm_Pitch1.27mm" H 2400 4000 60  0001 C CNN
@@
 AR Path="/58B5D98C/58B4BD43" Ref="U22"  Part="1"
 AR Path="/58B5EE77/58B4BD43" Ref="U29"  Part="1"
-F 0 "U22" H 2400 4550 60  0000 C CNN
+F 0 "U8" H 2400 4550 60  0000 C CNN
 F 1 "TPD4E1B06" H 2400 4950 60  0000 C CNN
 F 2 "TO_SOT_Packages_SMD:SC-70-6" H 2400 4750 60  0001 C CNN
@@
 AR Path="/58B5D98C/58B4BD4A" Ref="U26"  Part="1"
 AR Path="/58B5EE77/58B4BD4A" Ref="U33"  Part="1"
-F 0 "U26" H 2400 6750 60  0000 C CNN
+F 0 "U12" H 2400 6750 60  0000 C CNN
 F 1 "TPD4E1B06" H 2400 7150 60  0000 C CNN
 F 2 "TO_SOT_Packages_SMD:SC-70-6" H 2400 6950 60  0001 C CNN
@@
 AR Path="/58B5D98C/58B4BD51" Ref="U23"  Part="1"
 AR Path="/58B5EE77/58B4BD51" Ref="U30"  Part="1"
-F 0 "U23" H 2400 5100 60  0000 C CNN
+F 0 "U9" H 2400 5100 60  0000 C CNN
 F 1 "TPD4E1B06" H 2400 5500 60  0000 C CNN
 F 2 "TO_SOT_Packages_SMD:SC-70-6" H 2400 5300 60  0001 C CNN
@@
 AR Path="/58B5D98C/58B4BD58" Ref="U24"  Part="1"
 AR Path="/58B5EE77/58B4BD58" Ref="U31"  Part="1"
-F 0 "U24" H 2400 5650 60  0000 C CNN
+F 0 "U10" H 2400 5650 60  0000 C CNN
 F 1 "TPD4E1B06" H 2400 6050 60  0000 C CNN
 F 2 "TO_SOT_Packages_SMD:SC-70-6" H 2400 5850 60  0001 C CNN
@@
 AR Path="/58B5D98C/58B4BD5F" Ref="U25"  Part="1"
 AR Path="/58B5EE77/58B4BD5F" Ref="U32"  Part="1"
-F 0 "U25" H 2400 6200 60  0000 C CNN
+F 0 "U11" H 2400 6200 60  0000 C CNN
 F 1 "TPD4E1B06" H 2400 6600 60  0000 C CNN
 F 2 "TO_SOT_Packages_SMD:SC-70-6" H 2400 6400 60  0001 C CNN
@@
 AR Path="/58B5D98C/58B4EEE3" Ref="P3"  Part="1"
 AR Path="/58B5EE77/58B4EEE3" Ref="P4"  Part="1"
-F 0 "P3" H 4600 6550 50  0000 C CNN
+F 0 "P1" H 4600 6550 50  0000 C CNN
 F 1 "CONN_02X10" V 4600 6000 50  0000 C CNN
 F 2 "Pin_Headers:Pin_Header_Angled_2x10" H 4600 4800 50  0001 C CNN
@@
 Text Label 10150 2450 0    60   ~ 0
 IOVDD
+Text Label 4300 3100 0    60   ~ 0
+CONVST_SAR
+Text Label 4200 3100 2    60   ~ 0
+GND
+Wire Wire Line
+	4200 3100 4300 3100
 $EndSCHEMATC

Commit message: kicad
Parts:
- removed U12: TPD4E1B06, TO_SOT_Packages_SMD:SC-70-6, symbol TPD4E1B06
Connections:
- net VSS is gone; now on net GND: U10.3 (GND), U11.3 (GND), U8.3 (GND), U9.3 (GND)
- net GND: now also P1.19 (P19), P1.20 (P20)
- net at P1.1 (P1): now also P1.2 (P2)
Changed lines of the file:
@@
 EESchema Schematic File Version 2
-LIBS:FreeSmartEEG_AD7770_STM32F405VG_nRF52832_ESP8266-rescue
 LIBS:power
 LIBS:device
@@
 LIBS:valves
 LIBS:stm32f410rbt6
-LIBS:AD7768
 LIBS:esp8266
 LIBS:stm32f103r8t7
 LIBS:nrf52832
-LIBS:AD7779
 LIBS:STM32F405VG
 LIBS:AD7770
@@
 LIBS:473521001
 LIBS:adp7118aujz-3.3
+LIBS:tlv73333pdbvt
 LIBS:FreeEEG32-cache
 EELAYER 25 0
@@
 F 3 "" H 2400 4750 60  0001 C CNN
 	1    2400 4750
-	1    0    0    -1
-$EndComp
-$Comp
-L TPD4E1B06 U12
-U 1 1 58B4BD4A
-P 2400 6950
-AR Path="/58B4B6C8/58B4BD4A" Ref="U12"  Part="1"
-AR Path="/58B5BC1A/58B4BD4A" Ref="U19"  Part="1"
-AR Path="/58B5D98C/58B4BD4A" Ref="U26"  Part="1"
-AR Path="/58B5EE77/58B4BD4A" Ref="U33"  Part="1"
-F 0 "U12" H 2400 6750 60  0000 C CNN
-F 1 "TPD4E1B06" H 2400 7150 60  0000 C CNN
-F 2 "TO_SOT_Packages_SMD:SC-70-6" H 2400 6950 60  0001 C CNN
-F 3 "" H 2400 6950 60  0001 C CNN
-	1    2400 6950
 	1    0    0    -1
 $EndComp
@@
 Text Label 1950 3900 2    60   ~ 0
 V+
-Text Label 1950 4100 2    60   ~ 0
-GND
-Text Label 1950 7050 2    60   ~ 0
-VSS
-Text Label 1950 4850 2    60   ~ 0
-VSS
-Text Label 1950 5400 2    60   ~ 0
-VSS
-Text Label 1950 5950 2    60   ~ 0
-VSS
-Text Label 1950 6500 2    60   ~ 0
-VSS
 Text HLabel 1150 2000 0    60   Input ~ 0
 SYNC_OUT
@@
 	2850 4000 2800 4000
 Wire Wire Line
-	1950 7050 2000 7050
-Wire Wire Line
 	1950 4850 2000 4850
 Wire Wire Line
@@
 Text Label 4200 1900 2    60   ~ 0
 GND
-Text Label 10150 3500 0    60   ~ 0
-GND
-Text Label 10150 3700 0    60   ~ 0
-GND
-Text Label 10150 2900 0    60   ~ 0
-GND
-Text Label 10150 2600 0    60   ~ 0
-GND
 Text Label 10150 1900 0    60   ~ 0
 GND
@@
 GND
 Text Label 4200 2000 2    60   ~ 0
-AVDD
-Text Label 10150 3600 0    60   ~ 0
-AVDD
-Text Label 10150 2700 0    60   ~ 0
 AVDD
 Text Label 10150 2100 0    60   ~ 0
@@
 Text Label 7200 5100 0    60   ~ 0
 EPAD
-Text Label 7100 5100 2    60   ~ 0
-GND
 Wire Wire Line
 	7200 5100 7100 5100
@@
 Wire Wire Line
 	4200 3100 4300 3100
+Wire Wire Line
+	4300 6450 4350 6450
+Wire Wire Line
+	4900 6450 4850 6450
+Wire Wire Line
+	4850 5550 4850 5400
+Wire Wire Line
+	4850 5400 4350 5400
+Wire Wire Line
+	4350 5400 4350 5550
+Text Label 10150 3600 0    60   ~ 0
+AVDD
+Text Label 10150 2600 0    60   ~ 0
+GND
+Text Label 10150 2700 0    60   ~ 0
+AVDD
+Text Label 10150 2900 0    60   ~ 0
+GND
+Text Label 10150 3500 0    60   ~ 0
+GND
+Text Label 10150 3700 0    60   ~ 0
+GND
+Text Label 7100 5100 2    60   ~ 0
+GND
+Text Label 4900 6450 0    60   ~ 0
+GND
+Text Label 4300 6450 2    60   ~ 0
+GND
+Text Label 1950 6500 2    60   ~ 0
+GND
+Text Label 1950 5950 2    60   ~ 0
+GND
+Text Label 1950 5400 2    60   ~ 0
+GND
+Text Label 1950 4850 2    60   ~ 0
+GND
+Text Label 1950 4100 2    60   ~ 0
+GND
 $EndSCHEMATC

Commit message: kicad
Parts:
- C12, C13, C14, C15, C30, C31, C32, C33: manf# (none) -> GRM155R60J105KE19D
- C16, C17, C18, C19, C20, C22, C23, C26, C27, C28, C34: manf# (none) -> MC0402B104K160CT
- U10, U11, U8: manf# (none) -> TPD4E1B06DCKR

Commit message: kicad
Changed lines of the file:
@@
 LIBS:sn6501
 LIBS:da2303
-LIBS:CP2102N-A01-GQFN24
 LIBS:sp0503bahtg
-LIBS:MPU-6500
 LIBS:LP5912
 LIBS:STM32F427ZI_x
@@
 LIBS:tlv73333pdbvt
 LIBS:adum1402brwz
+LIBS:MPU-6500
+LIBS:CP2102N-A01-GQFN24
 LIBS:FreeEEG32-cache
 EELAYER 25 0
@@
 $Descr A4 11693 8268
 encoding utf-8
-Sheet 3 6
+Sheet 5 6
 Title ""
 Date ""
@@
 AR Path="/58B5D98C/58B4BBD1" Ref="C61"  Part="1"
 AR Path="/58B5EE77/58B4BBD1" Ref="C82"  Part="1"
-F 0 "C38" H 5510 3970 50  0000 L CNN
+F 0 "C82" H 5510 3970 50  0000 L CNN
 F 1 "1u" H 5510 3820 50  0000 L CNN
 F 2 "Capacitors_SMD:C_0402" H 5500 3900 50  0001 C CNN
@@
 AR Path="/58B5D98C/58B4BBD8" Ref="C65"  Part="1"
 AR Path="/58B5EE77/58B4BBD8" Ref="C86"  Part="1"
-F 0 "C43" H 5760 3970 50  0000 L CNN
+F 0 "C86" H 5760 3970 50  0000 L CNN
 F 1 "100n" H 5760 3820 50  0000 L CNN
 F 2 "Capacitors_SMD:C_0402" H 5750 3900 50  0001 C CNN
@@
 AR Path="/58B5D98C/58B4BBDF" Ref="C64"  Part="1"
 AR Path="/58B5EE77/58B4BBDF" Ref="C85"  Part="1"
-F 0 "C41" H 5760 3670 50  0000 L CNN
+F 0 "C85" H 5760 3670 50  0000 L CNN
 F 1 "100n" H 5760 3520 50  0000 L CNN
 F 2 "Capacitors_SMD:C_0402" H 5750 3600 50  0001 C CNN
@@
 AR Path="/58B5D98C/58B4BBE6" Ref="C60"  Part="1"
 AR Path="/58B5EE77/58B4BBE6" Ref="C81"  Part="1"
-F 0 "C37" H 5510 3670 50  0000 L CNN
+F 0 "C81" H 5510 3670 50  0000 L CNN
 F 1 "1u" H 5510 3520 50  0000 L CNN
 F 2 "Capacitors_SMD:C_0402" H 5500 3600 50  0001 C CNN
@@
 AR Path="/58B5D98C/58B4BBED" Ref="C63"  Part="1"
 AR Path="/58B5EE77/58B4BBED" Ref="C84"  Part="1"
-F 0 "C40" H 5760 2270 50  0000 L CNN
+F 0 "C84" H 5760 2270 50  0000 L CNN
 F 1 "100n" H 5760 2120 50  0000 L CNN
 F 2 "Capacitors_SMD:C_0402" H 5750 2200 50  0001 C CNN
@@
 AR Path="/58B5D98C/58B4BBF4" Ref="C59"  Part="1"
 AR Path="/58B5EE77/58B4BBF4" Ref="C80"  Part="1"
-F 0 "C36" H 5510 2270 50  0000 L CNN
+F 0 "C80" H 5510 2270 50  0000 L CNN
 F 1 "1u" H 5510 2120 50  0000 L CNN
 F 2 "Capacitors_SMD:C_0402" H 5500 2200 50  0001 C CNN
@@
 AR Path="/58B5D98C/58B4BBFB" Ref="C62"  Part="1"
 AR Path="/58B5EE77/58B4BBFB" Ref="C83"  Part="1"
-F 0 "C39" H 5760 1970 50  0000 L CNN
+F 0 "C83" H 5760 1970 50  0000 L CNN
 F 1 "100n" H 5760 1820 50  0000 L CNN
 F 2 "Capacitors_SMD:C_0402" H 5750 1900 50  0001 C CNN
@@
 AR Path="/58B5D98C/58B4BC02" Ref="C58"  Part="1"
 AR Path="/58B5EE77/58B4BC02" Ref="C79"  Part="1"
-F 0 "C35" H 5510 1970 50  0000 L CNN
+F 0 "C79" H 5510 1970 50  0000 L CNN
 F 1 "1u" H 5510 1820 50  0000 L CNN
 F 2 "Capacitors_SMD:C_0402" H 5500 1900 50  0001 C CNN
@@
 AR Path="/58B5D98C/58B4BC09" Ref="C66"  Part="1"
 AR Path="/58B5EE77/58B4BC09" Ref="C87"  Part="1"
-F 0 "C44" H 8560 3570 50  0000 L CNN
+F 0 "C87" H 8560 3570 50  0000 L CNN
 F 1 "100n" H 8560 3420 50  0000 L CNN
 F 2 "Capacitors_SMD:C_0402" H 8550 3500 50  0001 C CNN
@@
 AR Path="/58B5D98C/58B4BC10" Ref="C73"  Part="1"
 AR Path="/58B5EE77/58B4BC10" Ref="C94"  Part="1"
-F 0 "C51" H 8810 3570 50  0000 L CNN
+F 0 "C94" H 8810 3570 50  0000 L CNN
 F 1 "1u" H 8810 3420 50  0000 L CNN
 F 2 "Capacitors_SMD:C_0402" H 8800 3500 50  0001 C CNN
@@
 AR Path="/58B5D98C/58B4BC17" Ref="C74"  Part="1"
 AR Path="/58B5EE77/58B4BC17" Ref="C95"  Part="1"
-F 0 "C53" H 8810 3870 50  0000 L CNN
+F 0 "C95" H 8810 3870 50  0000 L CNN
 F 1 "1u" H 8810 3720 50  0000 L CNN
 F 2 "Capacitors_SMD:C_0402" H 8800 3800 50  0001 C CNN
@@
 AR Path="/58B5D98C/58B4BC1E" Ref="C67"  Part="1"
 AR Path="/58B5EE77/58B4BC1E" Ref="C88"  Part="1"
-F 0 "C45" H 8560 3870 50  0000 L CNN
+F 0 "C88" H 8560 3870 50  0000 L CNN
 F 1 "100n" H 8560 3720 50  0000 L CNN
 F 2 "Capacitors_SMD:C_0402" H 8550 3800 50  0001 C CNN
@@
 AR Path="/58B5D98C/58B4BC25" Ref="C78"  Part="1"
 AR Path="/58B5EE77/58B4BC25" Ref="C99"  Part="1"
-F 0 "C57" H 8910 3070 50  0000 L CNN
+F 0 "C99" H 8910 3070 50  0000 L CNN
 F 1 "100n" H 8910 2920 50  0000 L CNN
 F 2 "Capacitors_SMD:C_0402" H 8900 3000 50  0001 C CNN
@@
 AR Path="/58B5D98C/58B4BC2C" Ref="C68"  Part="1"
 AR Path="/58B5EE77/58B4BC2C" Ref="C89"  Part="1"
-F 0 "C46" H 8310 2920 50  0000 L CNN
+F 0 "C89" H 8310 2920 50  0000 L CNN
 F 1 "100n" H 8310 2770 50  0000 L CNN
 F 2 "Capacitors_SMD:C_0402" H 8300 2850 50  0001 C CNN
@@
 AR Path="/58B5D98C/58B4BC33" Ref="C71"  Part="1"
 AR Path="/58B5EE77/58B4BC33" Ref="C92"  Part="1"
-F 0 "C49" H 8660 2870 50  0000 L CNN
+F 0 "C92" H 8660 2870 50  0000 L CNN
 F 1 "100n" H 8660 2720 50  0000 L CNN
 F 2 "Capacitors_SMD:C_0402" H 8650 2800 50  0001 C CNN
@@
 AR Path="/58B5D98C/58B4BC3A" Ref="C70"  Part="1"
 AR Path="/58B5EE77/58B4BC3A" Ref="C91"  Part="1"
-F 0 "C48" H 8660 2070 50  0000 L CNN
+F 0 "C91" H 8660 2070 50  0000 L CNN
 F 1 "100n" H 8660 1920 50  0000 L CNN
 F 2 "Capacitors_SMD:C_0402" H 8650 2000 50  0001 C CNN
@@
 AR Path="/58B5D98C/58B4BC41" Ref="C72"  Part="1"
 AR Path="/58B5EE77/58B4BC41" Ref="C93"  Part="1"
-F 0 "C50" H 8310 2020 50  0000 L CNN
+F 0 "C93" H 8310 2020 50  0000 L CNN
 F 1 "100n" H 8310 1870 50  0000 L CNN
 F 2 "Capacitors_SMD:C_0402" H 8300 1950 50  0001 C CNN
@@
 AR Path="/58B5D98C/58B4BC48" Ref="C69"  Part="1"
 AR Path="/58B5EE77/58B4BC48" Ref="C90"  Part="1"
-F 0 "C47" H 8660 1770 50  0000 L CNN
+F 0 "C90" H 8660 1770 50  0000 L CNN
 F 1 "100n" H 8660 1620 50  0000 L CNN
 F 2 "Capacitors_SMD:C_0402" H 8650 1700 50  0001 C CNN
@@
 AR Path="/58B5D98C/58B4BC4F" Ref="C77"  Part="1"
 AR Path="/58B5EE77/58B4BC4F" Ref="C98"  Part="1"
-F 0 "C56" H 8910 2870 50  0000 L CNN
+F 0 "C98" H 8910 2870 50  0000 L CNN
 F 1 "1u" H 8910 2720 50  0000 L CNN
 F 2 "Capacitors_SMD:C_0402" H 8900 2800 50  0001 C CNN
@@
 AR Path="/58B5D98C/58B4BC56" Ref="C76"  Part="1"
 AR Path="/58B5EE77/58B4BC56" Ref="C97"  Part="1"
-F 0 "C55" H 8910 2070 50  0000 L CNN
+F 0 "C97" H 8910 2070 50  0000 L CNN
 F 1 "1u" H 8910 1920 50  0000 L CNN
 F 2 "Capacitors_SMD:C_0402" H 8900 2000 50  0001 C CNN
@@
 AR Path="/58B5D98C/58B4BC5D" Ref="C75"  Part="1"
 AR Path="/58B5EE77/58B4BC5D" Ref="C96"  Part="1"
-F 0 "C54" H 8910 1770 50  0000 L CNN
+F 0 "C96" H 8910 1770 50  0000 L CNN
 F 1 "1u" H 8910 1620 50  0000 L CNN
 F 2 "Capacitors_SMD:C_0402" H 8900 1700 50  0001 C CNN
@@
 AR Path="/58B5D98C/58B4BD09" Ref="U27"  Part="1"
 AR Path="/58B5EE77/58B4BD09" Ref="U34"  Part="1"
-F 0 "U20" H 7150 3100 60  0000 C CNN
+F 0 "U34" H 7150 3100 60  0000 C CNN
 F 1 "AD7770" H 7150 3000 60  0000 C CNN
 F 2 "Housings_DFN_QFN:QFN-64-1EP_9x9mm_Pitch0.5mm" H 7150 3050 60  0001 C CNN
@@
 AR Path="/58B5D98C/58B4BD10" Ref="U21"  Part="1"
 AR Path="/58B5EE77/58B4BD10" Ref="U28"  Part="1"
-F 0 "U14" H 2400 3700 60  0000 C CNN
+F 0 "U28" H 2400 3700 60  0000 C CNN
 F 1 "ADR4525" H 2400 4200 60  0000 C CNN
 F 2 "Housings_SOIC:SOIC-8_3.9x4.9mm_Pitch1.27mm" H 2400 4000 60  0001 C CNN
@@
 AR Path="/58B5D98C/58B4BD43" Ref="U22"  Part="1"
 AR Path="/58B5EE77/58B4BD43" Ref="U29"  Part="1"
-F 0 "U15" H 2400 4550 60  0000 C CNN
+F 0 "U29" H 2400 4550 60  0000 C CNN
 F 1 "TPD4E1B06" H 2400 4950 60  0000 C CNN
 F 2 "TO_SOT_Packages_SMD:SC-70-6" H 2400 4750 60  0001 C CNN
@@
 AR Path="/58B5D98C/58B4BD51" Ref="U23"  Part="1"
 AR Path="/58B5EE77/58B4BD51" Ref="U30"  Part="1"
-F 0 "U16" H 2400 5100 60  0000 C CNN
+F 0 "U30" H 2400 5100 60  0000 C CNN
 F 1 "TPD4E1B06" H 2400 5500 60  0000 C CNN
 F 2 "TO_SOT_Packages_SMD:SC-70-6" H 2400 5300 60  0001 C CNN
@@
 AR Path="/58B5D98C/58B4BD58" Ref="U24"  Part="1"
 AR Path="/58B5EE77/58B4BD58" Ref="U31"  Part="1"
-F 0 "U17" H 2400 5650 60  0000 C CNN
+F 0 "U31" H 2400 5650 60  0000 C CNN
 F 1 "TPD4E1B06" H 2400 6050 60  0000 C CNN
 F 2 "TO_SOT_Packages_SMD:SC-70-6" H 2400 5850 60  0001 C CNN
@@
 AR Path="/58B5D98C/58B4BD5F" Ref="U25"  Part="1"
 AR Path="/58B5EE77/58B4BD5F" Ref="U32"  Part="1"
-F 0 "U18" H 2400 6200 60  0000 C CNN
+F 0 "U32" H 2400 6200 60  0000 C CNN
 F 1 "TPD4E1B06" H 2400 6600 60  0000 C CNN
 F 2 "TO_SOT_Packages_SMD:SC-70-6" H 2400 6400 60  0001 C CNN
@@
 AR Path="/58B5D98C/58B4EEE3" Ref="P3"  Part="1"
 AR Path="/58B5EE77/58B4EEE3" Ref="P4"  Part="1"
-F 0 "P2" H 4600 6550 50  0000 C CNN
+F 0 "P4" H 4600 6550 50  0000 C CNN
 F 1 "CONN_02X10" V 4600 6000 50  0000 C CNN
 F 2 "Pin_Headers:Pin_Header_Angled_2x10" H 4600 4800 50  0001 C CNN

Commit message: kicad
Connections:
- net AVDD: now also P1.20 (P20)
- net GND: no longer P1.20 (P20)
Changed lines of the file:
@@
 Text Label 7100 5100 2    60   ~ 0
-GND
-Text Label 4900 6450 0    60   ~ 0
 GND
 Text Label 4300 6450 2    60   ~ 0
@@
 Text Label 1950 4100 2    60   ~ 0
 GND
+Text Label 4900 6450 0    60   ~ 0
+AVDD
 $EndSCHEMATC

Commit message: kicad
Parts:
- added C132: 10u, Capacitors_SMD:C_0603, symbol C_Small
- added C134, C145: 100n, Capacitors_SMD:C_0402, symbol C_Small
- added C135: 22u, Capacitors_SMD:C_0805, symbol C_Small
- added U4: TPD4E1B06, TO_SOT_Packages_SMD:SC-70-6, symbol TPD4E1B06
Connections:
- net AIN0+: now also U8.1 (IO1); no longer U8.5 (IO4)
- net AIN0-: now also U8.2 (IO2); no longer U8.4 (IO3)
- net AIN1+: now also U9.5 (IO4); no longer U8.1 (IO1)
- net AIN1-: now also U9.4 (IO3); no longer U8.2 (IO2)
- net AIN2+: now also U9.1 (IO1); no longer U9.5 (IO4)
- net AIN2-: now also U9.2 (IO2); no longer U9.4 (IO3)
- net AIN3+: now also U10.5 (IO4); no longer U9.1 (IO1)
- net AIN3-: now also U10.4 (IO3); no longer U9.2 (IO2)
- net AIN4+: now also U10.1 (IO1); no longer U10.5 (IO4)
- net AIN4-: now also U10.2 (IO2); no longer U10.4 (IO3)
- net AIN5+: now also U11.5 (IO4); no longer U10.1 (IO1)
- net AIN5-: now also U11.4 (IO3); no longer U10.2 (IO2)
- net AIN6+: now also U11.1 (IO1); no longer U11.5 (IO4)
- net AIN6-: now also U11.2 (IO2); no longer U11.4 (IO3)
- net AIN7+: now also U4.5 (IO4); no longer U11.1 (IO1)
- net AIN7-: now also U4.4 (IO3); no longer U11.2 (IO2)
- net AVDD: now also U4.1 (IO1)
- net GND: now also C132.1, C134.1, C135.1, C145.1, U4.3 (GND); no longer C12.2, C13.2, C16.2, C17.2, C20.1, C21.1, C22.2, C23.2, C26.1, C27.2, C28.1, C29.1, C30.1, C31.2, C32.1, C33.2, C34.1, P1.19 (P19), U13.42 (REF2-), U13.44 (AVSS1B), U13.5 (AVSS1A), U13.50 (AVSS2B), U13.53 (AVSS3), U13.60 (AVSS2A), U13.61 (AVSS4), U13.65 (EPAD), U13.7 (REF1-)
- net REF1+: now also C134.2, C135.2
- net V+: now also C132.2, C145.2
- net REF: now reaches P1.1 (P1), P1.2 (P2)
- net REF: now also U8.4 (IO3), U8.5 (IO4)
- new net AVSS: C12.2, C13.2, C16.2, C17.2, C20.1, C21.1, C22.2, C23.2, C26.1, C27.2, C28.1, C29.1, C30.1, C31.2, C32.1, C33.2, C34.1, P1.19 (P19), U13.42 (REF2-), U13.44 (AVSS1B), U13.5 (AVSS1A), U13.50 (AVSS2B), U13.53 (AVSS3), U13.60 (AVSS2A), U13.61 (AVSS4), U13.65 (EPAD), U13.7 (REF1-), U4.2 (IO2)
