File: KiCad/ADC.sch (KiCad schematic (older format))
At the start: 33 parts, among them P1 CONN_02X10, U10 TPD4E1B06, U11 TPD4E1B06, U13 AD7770, U4 TPD4E1B06, U7 ADR4525, U8 TPD4E1B06, U9 TPD4E1B06

Commit message: kicad
Connections:
- net AVDD: now also C132.2, C145.2, U7.2 (VIN)
- net AVSS: now also C132.1, C134.1, C135.1, C145.1, U7.4 (GND)
- net GND: no longer C132.1, C134.1, C135.1, C14.2, C145.1, C15.2, C18.2, C19.2, U13.17 (CONVST_SAR), U13.22 (DGND), U13.31 (XTAL1), U13.56 (CLK_SEL), U7.4 (GND)
- net V+: no longer C132.2, C145.2, U7.2 (VIN)
- net VCM: now also P1.2 (P2), U8.5 (IO4)
- net REF renamed AINREF
- net AINREF: no longer P1.2 (P2), U8.5 (IO4)
- new net DGND: C14.2, C15.2, C18.2, C19.2, U13.17 (CONVST_SAR), U13.22 (DGND), U13.31 (XTAL1), U13.56 (CLK_SEL)
Changed lines of the file:
@@
 EESchema Schematic File Version 2
+LIBS:FreeEEG32-rescue
 LIBS:power
 LIBS:device
@@
 LIBS:MPU-6500
 LIBS:CP2102N-A01-GQFN24
+LIBS:LSM6DS3
+LIBS:transformer_sp_ss
 LIBS:FreeEEG32-cache
 EELAYER 25 0
@@
 Text Label 8100 1500 0    60   ~ 0
 AUXAIN-
-Text Label 1500 3900 2    60   ~ 0
-V+
 Text HLabel 1150 2100 0    60   Input ~ 0
 SYNC_OUT
@@
 Text Label 10050 1700 2    60   ~ 0
 AVDD4
-Text Label 4300 3500 0    60   ~ 0
+Text Label 1250 3200 0    60   ~ 0
 DGND
 Text Label 4300 2200 0    60   ~ 0
@@
 Text Label 4300 1900 0    60   ~ 0
 AVSS1A
-Text Label 4200 3500 2    60   ~ 0
-GND
 Text Label 4200 2000 2    60   ~ 0
 AVDD
@@
 VREF
 Wire Wire Line
-	4300 3500 4200 3500
-Wire Wire Line
 	4300 2200 4200 2200
 Wire Wire Line
@@
 F 2 "Pin_Headers:Pin_Header_Angled_2x10" H 4600 4800 50  0001 C CNN
 F 3 "" H 4600 4800 50  0000 C CNN
-F 4 "PLD-10R" H 4600 6000 60  0000 C CNN "manf#"
+F 4 "PLD-10R" H 4600 6000 60  0001 C CNN "manf#"
 	1    4600 6000
 	1    0    0    -1
@@
 	4300 6350 4350 6350
 Wire Wire Line
-	4300 5550 4350 5550
-Wire Wire Line
-	4900 5550 4850 5550
+	4000 5550 4350 5550
+Wire Wire Line
+	5200 5550 4850 5550
 Wire Wire Line
 	4900 6350 4850 6350
@@
 Text Label 1950 4850 2    60   ~ 0
 GND
-Text Label 1500 4100 2    60   ~ 0
-GND
 Text Label 4900 6450 0    60   ~ 0
 AVDD
@@
 	3250 4000 3300 4000
 Connection ~ 3150 3900
-Text Label 3300 4100 0    60   ~ 0
-GND
 Wire Wire Line
 	2950 4100 3300 4100
@@
 Text Label 1950 6850 2    60   ~ 0
 AVDD
-Wire Wire Line
-	2850 4750 2850 4850
 Text GLabel 2850 4850 2    60   Input ~ 0
-REF
-Text GLabel 4900 5550 2    60   Input ~ 0
-REF
-Text GLabel 4300 5550 0    60   Input ~ 0
-REF
+AINREF
+Text GLabel 4000 5550 0    60   Input ~ 0
+AINREF
+Text Label 3300 4100 0    60   ~ 0
+AVSS
+Text Label 1500 4100 2    60   ~ 0
+AVSS
+Text HLabel 1150 3200 0    60   Input ~ 0
+DGND
+Wire Wire Line
+	1150 3200 1250 3200
+Text Label 5200 5550 0    60   ~ 0
+VCM
+Text Label 2850 4750 0    60   ~ 0
+VCM
+Text Label 1500 3900 2    60   ~ 0
+AVDD
 $EndSCHEMATC

Commit message: kicad
Changed lines of the file:
@@
 LIBS:LSM6DS3
 LIBS:transformer_sp_ss
+LIBS:sn6505b
 LIBS:FreeEEG32-cache
 EELAYER 25 0
@@
 AR Path="/58B5EE77/58B4BBD1" Ref="C82"  Part="1"
 AR Path="/58E92942/58B4BBD1" Ref="C38"  Part="1"
-F 0 "C61" H 5510 3970 50  0000 L CNN
+F 0 "C38" H 5510 3970 50  0000 L CNN
 F 1 "1u" H 5510 3820 50  0000 L CNN
 F 2 "Capacitors_SMD:C_0402" H 5500 3900 50  0001 C CNN
@@
 AR Path="/58B5EE77/58B4BBD8" Ref="C86"  Part="1"
 AR Path="/58E92942/58B4BBD8" Ref="C43"  Part="1"
-F 0 "C65" H 5760 3970 50  0000 L CNN
+F 0 "C43" H 5760 3970 50  0000 L CNN
 F 1 "100n" H 5760 3820 50  0000 L CNN
 F 2 "Capacitors_SMD:C_0402" H 5750 3900 50  0001 C CNN
@@
 AR Path="/58B5EE77/58B4BBDF" Ref="C85"  Part="1"
 AR Path="/58E92942/58B4BBDF" Ref="C41"  Part="1"
-F 0 "C64" H 5760 3670 50  0000 L CNN
+F 0 "C41" H 5760 3670 50  0000 L CNN
 F 1 "100n" H 5760 3520 50  0000 L CNN
 F 2 "Capacitors_SMD:C_0402" H 5750 3600 50  0001 C CNN
@@
 AR Path="/58B5EE77/58B4BBE6" Ref="C81"  Part="1"
 AR Path="/58E92942/58B4BBE6" Ref="C37"  Part="1"
-F 0 "C60" H 5510 3670 50  0000 L CNN
+F 0 "C37" H 5510 3670 50  0000 L CNN
 F 1 "1u" H 5510 3520 50  0000 L CNN
 F 2 "Capacitors_SMD:C_0402" H 5500 3600 50  0001 C CNN
@@
 AR Path="/58B5EE77/58B4BBED" Ref="C84"  Part="1"
 AR Path="/58E92942/58B4BBED" Ref="C40"  Part="1"
-F 0 "C63" H 5760 2270 50  0000 L CNN
+F 0 "C40" H 5760 2270 50  0000 L CNN
 F 1 "100n" H 5760 2120 50  0000 L CNN
 F 2 "Capacitors_SMD:C_0402" H 5750 2200 50  0001 C CNN
@@
 AR Path="/58B5EE77/58B4BBF4" Ref="C80"  Part="1"
 AR Path="/58E92942/58B4BBF4" Ref="C36"  Part="1"
-F 0 "C59" H 5510 2270 50  0000 L CNN
+F 0 "C36" H 5510 2270 50  0000 L CNN
 F 1 "1u" H 5510 2120 50  0000 L CNN
 F 2 "Capacitors_SMD:C_0402" H 5500 2200 50  0001 C CNN
@@
 AR Path="/58B5EE77/58B4BBFB" Ref="C83"  Part="1"
 AR Path="/58E92942/58B4BBFB" Ref="C39"  Part="1"
-F 0 "C62" H 5760 1970 50  0000 L CNN
+F 0 "C39" H 5760 1970 50  0000 L CNN
 F 1 "100n" H 5760 1820 50  0000 L CNN
 F 2 "Capacitors_SMD:C_0402" H 5750 1900 50  0001 C CNN
@@
 AR Path="/58B5EE77/58B4BC02" Ref="C79"  Part="1"
 AR Path="/58E92942/58B4BC02" Ref="C35"  Part="1"
-F 0 "C58" H 5510 1970 50  0000 L CNN
+F 0 "C35" H 5510 1970 50  0000 L CNN
 F 1 "1u" H 5510 1820 50  0000 L CNN
 F 2 "Capacitors_SMD:C_0402" H 5500 1900 50  0001 C CNN
@@
 AR Path="/58B5EE77/58B4BC09" Ref="C87"  Part="1"
 AR Path="/58E92942/58B4BC09" Ref="C44"  Part="1"
-F 0 "C66" H 8560 3570 50  0000 L CNN
+F 0 "C44" H 8560 3570 50  0000 L CNN
 F 1 "100n" H 8560 3420 50  0000 L CNN
 F 2 "Capacitors_SMD:C_0402" H 8550 3500 50  0001 C CNN
@@
 AR Path="/58B5EE77/58B4BC10" Ref="C94"  Part="1"
 AR Path="/58E92942/58B4BC10" Ref="C51"  Part="1"
-F 0 "C73" H 8810 3570 50  0000 L CNN
+F 0 "C51" H 8810 3570 50  0000 L CNN
 F 1 "1u" H 8810 3420 50  0000 L CNN
 F 2 "Capacitors_SMD:C_0402" H 8800 3500 50  0001 C CNN
@@
 AR Path="/58B5EE77/58B4BC17" Ref="C95"  Part="1"
 AR Path="/58E92942/58B4BC17" Ref="C53"  Part="1"
-F 0 "C74" H 8810 3870 50  0000 L CNN
+F 0 "C53" H 8810 3870 50  0000 L CNN
 F 1 "1u" H 8810 3720 50  0000 L CNN
 F 2 "Capacitors_SMD:C_0402" H 8800 3800 50  0001 C CNN
@@
 AR Path="/58B5EE77/58B4BC1E" Ref="C88"  Part="1"
 AR Path="/58E92942/58B4BC1E" Ref="C45"  Part="1"
-F 0 "C67" H 8560 3870 50  0000 L CNN
+F 0 "C45" H 8560 3870 50  0000 L CNN
 F 1 "100n" H 8560 3720 50  0000 L CNN
 F 2 "Capacitors_SMD:C_0402" H 8550 3800 50  0001 C CNN
@@
 AR Path="/58B5EE77/58B4BC25" Ref="C99"  Part="1"
 AR Path="/58E92942/58B4BC25" Ref="C57"  Part="1"
-F 0 "C78" H 8910 3070 50  0000 L CNN
+F 0 "C57" H 8910 3070 50  0000 L CNN
 F 1 "100n" H 8910 2920 50  0000 L CNN
 F 2 "Capacitors_SMD:C_0402" H 8900 3000 50  0001 C CNN
@@
 AR Path="/58B5EE77/58B4BC2C" Ref="C89"  Part="1"
 AR Path="/58E92942/58B4BC2C" Ref="C46"  Part="1"
-F 0 "C68" H 8310 2920 50  0000 L CNN
+F 0 "C46" H 8310 2920 50  0000 L CNN
 F 1 "100n" H 8310 2770 50  0000 L CNN
 F 2 "Capacitors_SMD:C_0402" H 8300 2850 50  0001 C CNN
@@
 AR Path="/58B5EE77/58B4BC33" Ref="C92"  Part="1"
 AR Path="/58E92942/58B4BC33" Ref="C49"  Part="1"
-F 0 "C71" H 8660 2870 50  0000 L CNN
+F 0 "C49" H 8660 2870 50  0000 L CNN
 F 1 "100n" H 8660 2720 50  0000 L CNN
 F 2 "Capacitors_SMD:C_0402" H 8650 2800 50  0001 C CNN
@@
 AR Path="/58B5EE77/58B4BC3A" Ref="C91"  Part="1"
 AR Path="/58E92942/58B4BC3A" Ref="C48"  Part="1"
-F 0 "C70" H 8660 2070 50  0000 L CNN
+F 0 "C48" H 8660 2070 50  0000 L CNN
 F 1 "100n" H 8660 1920 50  0000 L CNN
 F 2 "Capacitors_SMD:C_0402" H 8650 2000 50  0001 C CNN
@@
 AR Path="/58B5EE77/58B4BC41" Ref="C93"  Part="1"
 AR Path="/58E92942/58B4BC41" Ref="C50"  Part="1"
-F 0 "C72" H 8310 2020 50  0000 L CNN
+F 0 "C50" H 8310 2020 50  0000 L CNN
 F 1 "100n" H 8310 1870 50  0000 L CNN
 F 2 "Capacitors_SMD:C_0402" H 8300 1950 50  0001 C CNN
@@
 AR Path="/58B5EE77/58B4BC48" Ref="C90"  Part="1"
 AR Path="/58E92942/58B4BC48" Ref="C47"  Part="1"
-F 0 "C69" H 8660 1770 50  0000 L CNN
+F 0 "C47" H 8660 1770 50  0000 L CNN
 F 1 "100n" H 8660 1620 50  0000 L CNN
 F 2 "Capacitors_SMD:C_0402" H 8650 1700 50  0001 C CNN
@@
 AR Path="/58B5EE77/58B4BC4F" Ref="C98"  Part="1"
 AR Path="/58E92942/58B4BC4F" Ref="C56"  Part="1"
-F 0 "C77" H 8910 2870 50  0000 L CNN
+F 0 "C56" H 8910 2870 50  0000 L CNN
 F 1 "1u" H 8910 2720 50  0000 L CNN
 F 2 "Capacitors_SMD:C_0402" H 8900 2800 50  0001 C CNN
@@
 AR Path="/58B5EE77/58B4BC56" Ref="C97"  Part="1"
 AR Path="/58E92942/58B4BC56" Ref="C55"  Part="1"
-F 0 "C76" H 8910 2070 50  0000 L CNN
+F 0 "C55" H 8910 2070 50  0000 L CNN
 F 1 "1u" H 8910 1920 50  0000 L CNN
 F 2 "Capacitors_SMD:C_0402" H 8900 2000 50  0001 C CNN
@@
 AR Path="/58B5EE77/58B4BC5D" Ref="C96"  Part="1"
 AR Path="/58E92942/58B4BC5D" Ref="C54"  Part="1"
-F 0 "C75" H 8910 1770 50  0000 L CNN
+F 0 "C54" H 8910 1770 50  0000 L CNN
 F 1 "1u" H 8910 1620 50  0000 L CNN
 F 2 "Capacitors_SMD:C_0402" H 8900 1700 50  0001 C CNN
@@
 AR Path="/58B5EE77/58B4BD09" Ref="U34"  Part="1"
 AR Path="/58E92942/58B4BD09" Ref="U20"  Part="1"
-F 0 "U27" H 7150 3100 60  0000 C CNN
+F 0 "U20" H 7150 3100 60  0000 C CNN
 F 1 "AD7770" H 7150 3000 60  0000 C CNN
 F 2 "Housings_DFN_QFN:QFN-64-1EP_9x9mm_Pitch0.5mm" H 7150 3050 60  0001 C CNN
@@
 AR Path="/58B5EE77/58B4BD10" Ref="U28"  Part="1"
 AR Path="/58E92942/58B4BD10" Ref="U14"  Part="1"
-F 0 "U21" H 2400 3700 60  0000 C CNN
+F 0 "U14" H 2400 3700 60  0000 C CNN
 F 1 "ADR4525" H 2400 4200 60  0000 C CNN
 F 2 "Housings_SOIC:SOIC-8_3.9x4.9mm_Pitch1.27mm" H 2400 4000 60  0001 C CNN
@@
 AR Path="/58B5EE77/58B4BD43" Ref="U29"  Part="1"
 AR Path="/58E92942/58B4BD43" Ref="U15"  Part="1"
-F 0 "U22" H 2400 4550 60  0000 C CNN
+F 0 "U15" H 2400 4550 60  0000 C CNN
 F 1 "TPD4E1B06" H 2400 4950 60  0000 C CNN
 F 2 "TO_SOT_Packages_SMD:SC-70-6" H 2400 4750 60  0001 C CNN
@@
 AR Path="/58B5EE77/58B4BD51" Ref="U30"  Part="1"
 AR Path="/58E92942/58B4BD51" Ref="U16"  Part="1"
-F 0 "U23" H 2400 5100 60  0000 C CNN
+F 0 "U16" H 2400 5100 60  0000 C CNN
 F 1 "TPD4E1B06" H 2400 5500 60  0000 C CNN
 F 2 "TO_SOT_Packages_SMD:SC-70-6" H 2400 5300 60  0001 C CNN
@@
 AR Path="/58B5EE77/58B4BD58" Ref="U31"  Part="1"
 AR Path="/58E92942/58B4BD58" Ref="U17"  Part="1"
-F 0 "U24" H 2400 5650 60  0000 C CNN
+F 0 "U17" H 2400 5650 60  0000 C CNN
 F 1 "TPD4E1B06" H 2400 6050 60  0000 C CNN
 F 2 "TO_SOT_Packages_SMD:SC-70-6" H 2400 5850 60  0001 C CNN
@@
 AR Path="/58B5EE77/58B4BD5F" Ref="U32"  Part="1"
 AR Path="/58E92942/58B4BD5F" Ref="U18"  Part="1"
-F 0 "U25" H 2400 6200 60  0000 C CNN
+F 0 "U18" H 2400 6200 60  0000 C CNN
 F 1 "TPD4E1B06" H 2400 6600 60  0000 C CNN
 F 2 "TO_SOT_Packages_SMD:SC-70-6" H 2400 6400 60  0001 C CNN
@@
 AR Path="/58B5EE77/58B4EEE3" Ref="P4"  Part="1"
 AR Path="/58E92942/58B4EEE3" Ref="P2"  Part="1"
-F 0 "P3" H 4600 6550 50  0000 C CNN
+F 0 "P2" H 4600 6550 50  0000 C CNN
 F 1 "CONN_02X10" V 4600 6000 50  0000 C CNN
 F 2 "Pin_Headers:Pin_Header_Angled_2x10" H 4600 4800 50  0001 C CNN
@@
 AR Path="/58B4B6C8/58E71F17" Ref="C141"  Part="1"
 AR Path="/58E92942/58E71F17" Ref="C137"  Part="1"
-F 0 "C133" H 1860 4070 50  0000 L CNN
+F 0 "C137" H 1860 4070 50  0000 L CNN
 F 1 "100n" H 1860 3920 50  0000 L CNN
 F 2 "Capacitors_SMD:C_0402" H 1850 4000 50  0001 C CNN
@@
 AR Path="/58B5EE77/58E7219F" Ref="C146"  Part="1"
 AR Path="/58E92942/58E7219F" Ref="C138"  Part="1"
-F 0 "C134" H 2960 4070 50  0000 L CNN
+F 0 "C138" H 2960 4070 50  0000 L CNN
 F 1 "100n" H 2960 3920 50  0000 L CNN
 F 2 "Capacitors_SMD:C_0402" H 2950 4000 50  0001 C CNN
@@
 AR Path="/58B5EE77/58E72DF6" Ref="C144"  Part="1"
 AR Path="/58E92942/58E72DF6" Ref="C136"  Part="1"
-F 0 "C132" H 1660 4070 50  0000 L CNN
+F 0 "C136" H 1660 4070 50  0000 L CNN
 F 1 "10u" H 1660 3920 50  0000 L CNN
 F 2 "Capacitors_SMD:C_0603" H 1650 4000 50  0001 C CNN
@@
 AR Path="/58B5EE77/58E72F8D" Ref="C147"  Part="1"
 AR Path="/58E92942/58E72F8D" Ref="C139"  Part="1"
-F 0 "C135" H 3160 4070 50  0000 L CNN
+F 0 "C139" H 3160 4070 50  0000 L CNN
 F 1 "22u" H 3160 3920 50  0000 L CNN
 F 2 "Capacitors_SMD:C_0805" H 3150 4000 50  0001 C CNN
@@
 AR Path="/58B5D98C/58ED7D80" Ref="U33"  Part="1"
 AR Path="/58B4B6C8/58ED7D80" Ref="U38"  Part="1"
-F 0 "U33" H 2400 6750 60  0000 C CNN
+F 0 "U4" H 2400 6750 60  0000 C CNN
 F 1 "TPD4E1B06" H 2400 7150 60  0000 C CNN
 F 2 "TO_SOT_Packages_SMD:SC-70-6" H 2400 6950 60  0001 C CNN
