File: KiCad/ISO_WIFI_USB.sch (KiCad schematic (older format))
At the start: 34 parts, among them P5 CONN_01X02, P6 CONN_01X06, P7 CONN_01X06, P8 USB_B, SW2 SWITCH_INV, SW3 SWITCH_INV, T1 da2303, U35 ISO7342c_uart, U36 ISO7341c_spi, U38 LP5907_WIFI, U40 CP2102N-24, U41 MPU-6500, U42 LP5912, U5 ESP-12E, U6 SN6505A

Commit message: kicad
Parts:
- U5: value ESP-12E -> ESP-12F; manf# ESP-12E -> ESP-12F
Connections:
- net labels removed: USART6_CTS, USART6_RTS, USART6_RX, USART6_TX
Other:
- moved on the sheet: C116, C117
Changed lines of the file:
@@
 P 7050 3300
 F 0 "U5" H 7050 3300 60  0000 C CNN
-F 1 "ESP-12E" H 7050 3500 60  0000 C CNN
+F 1 "ESP-12F" H 7050 3500 60  0000 C CNN
 F 2 "ESP-12E:ESP-12E" H 7050 3500 60  0001 C CNN
 F 3 "" H 7050 3500 60  0001 C CNN
-F 4 "ESP-12E" H 7050 3300 60  0000 C CNN "manf#"
+F 4 "ESP-12F" H 7050 3300 60  0000 C CNN "manf#"
 	1    7050 3300
 	1    0    0    -1
@@
 L LP5912 U42
 U 1 1 58D0BFCA
-P 7050 1750
-F 0 "U42" H 7050 1800 60  0000 C CNN
-F 1 "LP5912" H 7050 2000 60  0000 C CNN
-F 2 "WSON-6_2x2mm_Pitch0.65mm:WSON-6_2x2mm_Pitch0.65mm" H 7050 1750 60  0001 C CNN
-F 3 "" H 7050 1750 60  0001 C CNN
-	1    7050 1750
+P 6900 -650
+F 0 "U42" H 6900 -600 60  0000 C CNN
+F 1 "LP5912" H 6900 -400 60  0000 C CNN
+F 2 "WSON-6_2x2mm_Pitch0.65mm:WSON-6_2x2mm_Pitch0.65mm" H 6900 -650 60  0001 C CNN
+F 3 "" H 6900 -650 60  0001 C CNN
+	1    6900 -650
 	1    0    0    -1
 $EndComp
@@
 L C_Small C117
 U 1 1 58D0D29E
-P 7700 1700
-F 0 "C117" H 7710 1770 50  0000 L CNN
-F 1 "1u" H 7710 1620 50  0000 L CNN
-F 2 "Capacitors_SMD:C_0402" H 7700 1700 50  0001 C CNN
-F 3 "" H 7700 1700 50  0000 C CNN
-	1    7700 1700
+P 7550 -700
+F 0 "C117" H 7560 -630 50  0000 L CNN
+F 1 "1u" H 7560 -780 50  0000 L CNN
+F 2 "Capacitors_SMD:C_0402" H 7550 -700 50  0001 C CNN
+F 3 "" H 7550 -700 50  0000 C CNN
+	1    7550 -700
 	1    0    0    1
 $EndComp
@@
 L C_Small C116
 U 1 1 58D0D357
-P 6400 1700
-F 0 "C116" H 6410 1770 50  0000 L CNN
-F 1 "10u" H 6410 1620 50  0000 L CNN
-F 2 "Capacitors_SMD:C_0402" H 6400 1700 50  0001 C CNN
-F 3 "" H 6400 1700 50  0000 C CNN
-	1    6400 1700
+P 6250 -700
+F 0 "C116" H 6260 -630 50  0000 L CNN
+F 1 "10u" H 6260 -780 50  0000 L CNN
+F 2 "Capacitors_SMD:C_0402" H 6250 -700 50  0001 C CNN
+F 3 "" H 6250 -700 50  0000 C CNN
+	1    6250 -700
 	1    0    0    1
 $EndComp
-Text GLabel 7850 1750 2    60   Input ~ 0
+Text GLabel 7700 -650 2    60   Input ~ 0
 GND_WIFI
-Text GLabel 7850 1650 2    60   Input ~ 0
+Text GLabel 7700 -750 2    60   Input ~ 0
 V+_WIFI
-Text GLabel 6250 1750 0    60   Input ~ 0
+Text GLabel 6100 -650 0    60   Input ~ 0
 GND_WIFI
-Text GLabel 6250 1650 0    60   Input ~ 0
+Text GLabel 6100 -750 0    60   Input ~ 0
 VCC_WIFI
 Wire Wire Line
-	6250 1750 6300 1750
-Wire Wire Line
-	6300 1750 6300 1800
-Wire Wire Line
-	6300 1800 6500 1800
-Wire Wire Line
-	6250 1650 6300 1650
-Wire Wire Line
-	6300 1650 6300 1600
-Wire Wire Line
-	6300 1600 6500 1600
-Wire Wire Line
-	6500 1600 6500 1650
-Wire Wire Line
-	6500 1650 6550 1650
-Connection ~ 6400 1600
-Wire Wire Line
-	7550 1650 7600 1650
-Wire Wire Line
-	7600 1650 7600 1600
-Wire Wire Line
-	7600 1600 7800 1600
-Wire Wire Line
-	7800 1600 7800 1650
-Wire Wire Line
-	7800 1650 7850 1650
-Connection ~ 7700 1600
-Wire Wire Line
-	7850 1750 7800 1750
-Wire Wire Line
-	7800 1750 7800 1800
-Wire Wire Line
-	7800 1800 7600 1800
-Wire Wire Line
-	7600 1800 7600 1750
-Wire Wire Line
-	7600 1750 7550 1750
-Connection ~ 7700 1800
-Wire Wire Line
-	6500 1800 6500 1750
-Wire Wire Line
-	6500 1750 6550 1750
-Connection ~ 6400 1800
-Wire Wire Line
-	7050 2150 6400 2150
-Wire Wire Line
-	6400 2150 6400 1800
-Text GLabel 5400 6050 2    60   Input ~ 0
-USART6_RX
-Text GLabel 5400 6250 2    60   Input ~ 0
-USART6_TX
-Text GLabel 5400 6350 2    60   Input ~ 0
-USART6_RTS
-Text GLabel 5400 6150 2    60   Input ~ 0
-USART6_CTS
+	6100 -650 6150 -650
+Wire Wire Line
+	6150 -650 6150 -600
+Wire Wire Line
+	6150 -600 6350 -600
+Wire Wire Line
+	6100 -750 6150 -750
+Wire Wire Line
+	6150 -750 6150 -800
+Wire Wire Line
+	6150 -800 6350 -800
+Wire Wire Line
+	6350 -800 6350 -750
+Wire Wire Line
+	6350 -750 6400 -750
+Connection ~ 6250 -800
+Wire Wire Line
+	7400 -750 7450 -750
+Wire Wire Line
+	7450 -750 7450 -800
+Wire Wire Line
+	7450 -800 7650 -800
+Wire Wire Line
+	7650 -800 7650 -750
+Wire Wire Line
+	7650 -750 7700 -750
+Connection ~ 7550 -800
+Wire Wire Line
+	7700 -650 7650 -650
+Wire Wire Line
+	7650 -650 7650 -600
+Wire Wire Line
+	7650 -600 7450 -600
+Wire Wire Line
+	7450 -600 7450 -650
+Wire Wire Line
+	7450 -650 7400 -650
+Connection ~ 7550 -600
+Wire Wire Line
+	6350 -600 6350 -650
+Wire Wire Line
+	6350 -650 6400 -650
+Connection ~ 6250 -600
+Wire Wire Line
+	6900 -250 6250 -250
+Wire Wire Line
+	6250 -250 6250 -600
 Text GLabel 3000 900  2    60   Input ~ 0
 SPI6_SCK

Commit message: kicad
Parts:
- removed C116: 10u, Capacitors_SMD:C_0402, symbol C_Small
- removed C117: 1u, Capacitors_SMD:C_0402, symbol C_Small
- removed P5: CONN_01X02, Socket_Strips:Socket_Strip_Straight_1x02, symbol CONN_01X02
- removed P6, P7: CONN_01X06, Socket_Strips:Socket_Strip_Straight_1x06, symbol CONN_01X06
- removed R2: 1k, Resistors_SMD:R_0402, symbol R_Small
- removed SW2: SWITCH_INV, Buttons_Switches_SMD:SW_SPDT_PCM12, symbol SWITCH_INV
- removed U38: LP5907_WIFI, TO_SOT_Packages_SMD:SOT-23-5, symbol LP5907
- removed U41: MPU-6500, Housings_DFN_QFN:QFN-24-1EP_4x4mm_Pitch0.5mm, symbol MPU-6500
- removed U42: LP5912, WSON-6_2x2mm_Pitch0.65mm:WSON-6_2x2mm_Pitch0.65mm, symbol LP5912
- added P6, P7: CONN_02X03, Socket_Strips:Socket_Strip_Straight_2x03, symbol CONN_02X03
- added U19: TLV73333PDBVT, TO_SOT_Packages_SMD:SOT-23-5, symbol TLV73333PDBVT
- C111, C112: footprint Capacitors_SMD:C_0402 -> Capacitors_SMD:C_0603; manf# (none) -> GRM188R60J475KE19D
- C113, C114: footprint Capacitors_SMD:C_0402 -> Capacitors_SMD:C_0603; manf# (none) -> GRM188R61A106KE69D
- C24: value 1u -> 100n
- SW3: footprint Buttons_Switches_SMD:SW_SPDT_PCM12 -> Buttons_Switches_SMD:SW_SPST_B3U-1100P-B
Connections:
- net labels added: BOOT_WIFI, VDD_USB
- net labels removed: CH_PD_WIFI, SPI6_MISO, SPI6_MOSI, SPI6_NSS, SPI6_SCK
- wire segments 207 -> 179
Other:
- moved on the sheet: C107, C108, C113, C114, C115, C24, C25, C42, C52, D1, T1, U35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

Commit message: kicad
Parts:
- removed U35: ISO7342c_uart, Housings_SOIC:SOIC-16_7.5x10.3mm_Pitch1.27mm, symbol ISO7342c
- added U35: ADUM1402BRWZ, symbol ADUM1402BRWZ
- C107, C108, C109, C110, C115, C24, C42, C52: manf# (none) -> MC0402B104K160CT
- C25: manf# (none) -> GRM155R60J105KE19D
- P6, P7: manf# (none) -> PBD-3
- T1: manf# DA2303-ALD -> DA2303
Other:
- moved on the sheet: C113, C114, C115, D1, D2, T1, U6

Commit message: kicad
Changed lines of the file:
@@
 F 2 "TO_SOT_Packages_SMD:SOT-23-5" H 7000 1000 60  0001 C CNN
 F 3 "" H 7000 1000 60  0001 C CNN
-F 4 "TLV73333PDBVT" H 7000 1000 60  0000 C CNN "manf#"
+F 4 "TLV73333PDBVT" H 7000 1000 60  0001 C CNN "manf#"
 	1    7000 1000
 	1    0    0    -1

Commit message: kicad
Parts:
- U35: footprint (none) -> Housings_SOIC:SOIC-16_7.5x10.3mm_Pitch1.27mm
- U40: value CP2102N-24 -> CP2102N-A01-GQFN24
Changed lines of the file:
@@
 LIBS:sn6501
 LIBS:da2303
-LIBS:CP2102N-A01-GQFN24
 LIBS:sp0503bahtg
-LIBS:MPU-6500
 LIBS:LP5912
 LIBS:STM32F427ZI_x
@@
 LIBS:tlv73333pdbvt
 LIBS:adum1402brwz
+LIBS:MPU-6500
+LIBS:CP2102N-A01-GQFN24
 LIBS:FreeEEG32-cache
 EELAYER 25 0
@@
 Text GLabel 6350 3600 0    60   Input ~ 0
 UART_CTS_WIFI
-$Comp
-L CP2102N-A01-GQFN24_2sides U?
-U 1 1 58CE6FF7
-P 3650 3500
-AR Path="/58CE6FF7" Ref="U?"  Part="1"
-AR Path="/58CE50D0/58CE6FF7" Ref="U40"  Part="1"
-F 0 "U40" H 3650 3500 60  0000 C CNN
-F 1 "CP2102N-24" H 3650 4150 60  0000 C CNN
-F 2 "Housings_DFN_QFN:QFN-24-1EP_4x4mm_Pitch0.5mm" H 3050 4050 60  0001 C CNN
-F 3 "" H 3050 4050 60  0001 C CNN
-F 4 "CP2102N-A01-GQFN24" H 3650 3500 60  0001 C CNN "manf#"
-	1    3650 3500
-	1    0    0    -1
-$EndComp
 Text GLabel 4300 3350 2    60   Input ~ 0
 UART_RX_USB
@@
 F 0 "U35" H 4500 6200 60  0000 C CNN
 F 1 "ADUM1402BRWZ" H 4500 6650 60  0000 C CNN
-F 2 "" H 4500 6050 60  0001 C CNN
+F 2 "Housings_SOIC:SOIC-16_7.5x10.3mm_Pitch1.27mm" H 4500 6050 60  0001 C CNN
 F 3 "" H 4500 6050 60  0001 C CNN
 F 4 "ADUM1402BRWZ" H 4500 6200 60  0001 C CNN "manf#"
@@
 	1    0    0    -1
 $EndComp
+$Comp
+L CP2102N-A01-GQFN24_2sides U40
+U 1 1 58E30304
+P 3650 3500
+F 0 "U40" H 3650 3500 60  0000 C CNN
+F 1 "CP2102N-A01-GQFN24" H 3650 4150 60  0000 C CNN
+F 2 "Housings_DFN_QFN:QFN-24-1EP_4x4mm_Pitch0.5mm" H 3050 4050 60  0001 C CNN
+F 3 "" H 3050 4050 60  0001 C CNN
+F 4 "CP2102N-A01-GQFN24" H 3650 3500 60  0001 C CNN "manf#"
+	1    3650 3500
+	1    0    0    -1
+$EndComp

Commit message: kicad
Parts:
- removed SW3: SWITCH_INV, Buttons_Switches_SMD:SW_SPST_B3U-1100P-B, symbol SWITCH_INV
- added C126, C127: 100n, Capacitors_SMD:C_0402, symbol C_Small
- added R4, R5, R6: 47k, Resistors_SMD:R_0402, symbol R_Small
- added SW3: BOOT0, Buttons_Switches_SMD:SW_SPST_B3U-3000P-B, symbol SW_PUSH_SMALL
- added SW4: BOOT_WIFI, Buttons_Switches_SMD:SW_SPST_B3U-1000P, symbol SW_PUSH_SMALL
Connections:
- net GND_ISO_UART: now also C126.2, C127.2, R6.1, SW3.2, SW4.2
- net UART_RTS_USB: now also R6.2
- net VCC_WIFI: now also R4.1, R5.1; no longer U5.3 (CH_PD)
- net BOOT_WIFI: no longer names the net of U5.18 (GPIO0)
- net BOOT_WIFI: now also C127.1, R5.2, SW4.1
- new net: C126.1, R4.2, SW3.1, U5.3 (CH_PD)
Changed lines of the file:
@@
 Text GLabel 7750 3700 2    60   Input ~ 0
 GND_WIFI
-Text GLabel 7750 3600 2    60   Input ~ 0
+Text GLabel 8350 3600 2    60   Input ~ 0
 UART_RTS_WIFI
 Text GLabel 6350 3600 0    60   Input ~ 0
@@
 	6350 3600 6400 3600
 Wire Wire Line
-	7700 3600 7750 3600
+	7700 3600 8350 3600
 Wire Wire Line
 	4250 3350 4300 3350
@@
 Text GLabel 3000 3350 0    60   Input ~ 0
 VIO_USB
-Text GLabel 6350 3200 0    60   Input ~ 0
-VCC_WIFI
-Wire Wire Line
-	6350 3200 6400 3200
 $Comp
 L C_Small C115
@@
 Text GLabel 7750 3500 2    60   Input ~ 0
 VCC_WIFI
-Text GLabel 7750 3400 2    60   Input ~ 0
-BOOT_WIFI
 Wire Wire Line
 	7700 3500 7750 3500
-Wire Wire Line
-	7700 3400 7750 3400
-Text GLabel 7400 1500 2    60   Input ~ 0
+Text GLabel 8400 3400 2    60   Input ~ 0
 VCC_WIFI
-Text GLabel 6300 1600 0    60   Input ~ 0
+Text GLabel 8150 3200 2    60   Input ~ 0
 GND_WIFI
-Text GLabel 7400 1700 2    60   Input ~ 0
-BOOT_WIFI
-$Comp
-L SWITCH_INV SW3
-U 1 1 58E05F38
-P 6850 1600
-F 0 "SW3" H 6650 1750 50  0000 C CNN
-F 1 "SWITCH_INV" H 6700 1450 50  0000 C CNN
-F 2 "Buttons_Switches_SMD:SW_SPST_B3U-1100P-B" H 6850 1600 50  0001 C CNN
-F 3 "" H 6850 1600 50  0000 C CNN
-	1    6850 1600
-	1    0    0    -1
-$EndComp
-Wire Wire Line
-	6300 1600 6350 1600
-Wire Wire Line
-	7350 1500 7400 1500
-Wire Wire Line
-	7350 1700 7400 1700
 Wire Wire Line
 	9150 5400 9050 5400
@@
 	1    0    0    -1
 $EndComp
+$Comp
+L R_Small R5
+U 1 1 58E54546
+P 8250 3400
+F 0 "R5" H 8280 3420 50  0000 L CNN
+F 1 "47k" H 8280 3360 50  0000 L CNN
+F 2 "Resistors_SMD:R_0402" H 8250 3400 50  0001 C CNN
+F 3 "" H 8250 3400 50  0000 C CNN
+F 4 "RC0402FR-0747KL" H 8250 3400 60  0001 C CNN "manf#"
+	1    8250 3400
+	0    1    -1   0
+$EndComp
+$Comp
+L SW_PUSH_SMALL SW4
+U 1 1 58E5454F
+P 8000 3300
+F 0 "SW4" H 8150 3410 50  0000 C CNN
+F 1 "BOOT_WIFI" H 8000 3221 50  0000 C CNN
+F 2 "Buttons_Switches_SMD:SW_SPST_B3U-1000P" H 8000 3300 50  0001 C CNN
+F 3 "" H 8000 3300 50  0000 C CNN
+F 4 "B3U3000PMB" H 8000 3300 60  0001 C CNN "manf#"
+	1    8000 3300
+	0    -1   -1   0
+$EndComp
+$Comp
+L C_Small C127
+U 1 1 58E54F0F
+P 7800 3300
+F 0 "C127" H 7810 3370 50  0000 L CNN
+F 1 "100n" H 7810 3220 50  0000 L CNN
+F 2 "Capacitors_SMD:C_0402" H 7800 3300 50  0001 C CNN
+F 3 "" H 7800 3300 50  0000 C CNN
+F 4 "MC0402B104K160CT" H 7800 3300 60  0001 C CNN "manf#"
+	1    7800 3300
+	1    0    0    1
+$EndComp
+Wire Wire Line
+	7700 3400 8150 3400
+Connection ~ 7800 3400
+Connection ~ 7900 3400
+Wire Wire Line
+	8350 3400 8400 3400
+Wire Wire Line
+	7800 3200 8150 3200
+Connection ~ 8100 3200
+Text GLabel 5700 3200 0    60   Input ~ 0
+VCC_WIFI
+Text GLabel 5950 3000 0    60   Input ~ 0
+GND_WIFI
+$Comp
+L R_Small R4
+U 1 1 58E56B55
+P 5850 3200
+F 0 "R4" H 5880 3220 50  0000 L CNN
+F 1 "47k" H 5880 3160 50  0000 L CNN
+F 2 "Resistors_SMD:R_0402" H 5850 3200 50  0001 C CNN
+F 3 "" H 5850 3200 50  0000 C CNN
+F 4 "RC0402FR-0747KL" H 5850 3200 60  0001 C CNN "manf#"
+	1    5850 3200
+	0    -1   -1   0
+$EndComp
+$Comp
+L SW_PUSH_SMALL SW3
+U 1 1 58E56B5C
+P 6100 3100
+F 0 "SW3" H 6250 3210 50  0000 C CNN
+F 1 "BOOT0" H 6100 3021 50  0000 C CNN
+F 2 "Buttons_Switches_SMD:SW_SPST_B3U-3000P-B" H 6100 3100 50  0001 C CNN
+F 3 "" H 6100 3100 50  0000 C CNN
+F 4 "B3U1000P" H 6100 3100 60  0001 C CNN "manf#"
+	1    6100 3100
+	0    1    -1   0
+$EndComp
+$Comp
+L C_Small C126
+U 1 1 58E56B64
+P 6300 3100
+F 0 "C126" H 6310 3170 50  0000 L CNN
+F 1 "100n" H 6310 3020 50  0000 L CNN
+F 2 "Capacitors_SMD:C_0402" H 6300 3100 50  0001 C CNN
+F 3 "" H 6300 3100 50  0000 C CNN
+F 4 "MC0402B104K160CT" H 6300 3100 60  0001 C CNN "manf#"
+	1    6300 3100
+	-1   0    0    1
+$EndComp
+Wire Wire Line
+	6400 3200 5950 3200
+Connection ~ 6300 3200
+Connection ~ 6200 3200
+Wire Wire Line
+	5750 3200 5700 3200
+Wire Wire Line
+	6300 3000 5950 3000
+Connection ~ 6000 3000
+$Comp
+L R_Small R6
+U 1 1 58E572B8
+P 8350 3700
+F 0 "R6" H 8380 3720 50  0000 L CNN
+F 1 "47k" H 8380 3660 50  0000 L CNN
+F 2 "Resistors_SMD:R_0402" H 8350 3700 50  0001 C CNN
+F 3 "" H 8350 3700 50  0000 C CNN
+F 4 "RC0402FR-0747KL" H 8350 3700 60  0001 C CNN "manf#"
+	1    8350 3700
+	0    1    -1   0
+$EndComp
+Text GLabel 8500 3700 2    60   Input ~ 0
+GND_WIFI
+Wire Wire Line
+	8500 3700 8450 3700
+Wire Wire Line
+	8250 3600 8250 3700
+Connection ~ 8250 3600
 $EndSCHEMATC

Commit message: kicad
Parts:
- T1: manf# DA2303 -> DA2303-ALD
Changed lines of the file:
@@
 F 2 "SMT_Power_Transformer:SMT Power Transformer" H 8350 5000 50  0001 C CNN
 F 3 "" H 8350 5000 50  0000 C CNN
-F 4 "DA2303" H 8350 5000 60  0001 C CNN "manf#"
+F 4 "DA2303-ALD" H 8350 5000 60  0001 C CNN "manf#"
 	1    8350 5000
 	1    0    0    -1
