File: KiCad/ISO_WIFI_USB.sch (KiCad schematic (older format))
At the start: 33 parts, among them P6 CONN_02X03, P7 CONN_02X03, P8 USB_B, SW3 BOOT0, SW4 BOOT_WIFI, T1 da2303, U19 TLV73333PDBVT, U35 ADUM1402BRWZ, U36 ISO7341c_spi, U40 CP2102N-A01-GQFN24, U5 ESP-12F, U6 SN6505A

Commit message: kicad
Parts:
- P8: symbol USB_B -> USB_B-RESCUE-FreeEEG32
- SW3: manf# B3U1000P -> B3U-1000P
- SW4: manf# B3U3000PMB -> B3U-3000PM-B
- T1: footprint SMT_Power_Transformer:SMT Power Transformer -> da2303:da2303

Commit message: kicad
Parts:
- removed U6: SN6505A, TO_SOT_Packages_SMD:SOT-23-6, symbol SN6505A
- added U6: SN6505B, TO_SOT_Packages_SMD:SOT-23-6, symbol SN6505B
Connections:
- net GND_ISO_UART: now also U6.4 (GND)
- net V+_ISO_UART: now also U6.2 (VCC), U6.5 (EN)
- net at T1.4 (IN2B): now also U6.1 (D1)
- net at T1.1 (IN1A): now also U6.3 (D2)
Changed lines of the file:
@@
 LIBS:LSM6DS3
 LIBS:transformer_sp_ss
+LIBS:sn6505b
 LIBS:FreeEEG32-cache
 EELAYER 25 0
@@
 Text GLabel 1250 6100 0    60   Input ~ 0
 V+_ISO_UART
-$Comp
-L SN6505A U6
-U 1 1 58CE6FCD
-P 7150 5000
-F 0 "U6" H 7150 4800 60  0000 C CNN
-F 1 "SN6505A" H 7150 5200 60  0000 C CNN
-F 2 "TO_SOT_Packages_SMD:SOT-23-6" H 7150 5000 60  0001 C CNN
-F 3 "" H 7150 5000 60  0000 C CNN
-F 4 "SN6505ADBVT" H 7150 5000 60  0001 C CNN "manf#"
-	1    7150 5000
-	-1   0    0    1
-$EndComp
 $Comp
 L D_Schottky_Small D1
@@
 	1    0    0    -1
 $EndComp
+$Comp
+L SN6505B U6
+U 1 1 58EE714E
+P 7150 5000
+F 0 "U6" H 7150 4800 60  0000 C CNN
+F 1 "SN6505B" H 7150 5200 60  0000 C CNN
+F 2 "TO_SOT_Packages_SMD:SOT-23-6" H 7150 5000 60  0001 C CNN
+F 3 "" H 7150 5000 60  0000 C CNN
+F 4 "SN6505BDBVT" H 7150 5000 60  0001 C CNN "manf#"
+	1    7150 5000
+	-1   0    0    1
+$EndComp
 $EndSCHEMATC
